Commit message: Add materials again, update joint limits:

File: pal_pro_gripper_description/urdf/materials.urdf.xacro (robot description, xacro)
@@ -8,9 +8,9 @@
 -->
 <robot>
-  <!-- <material name="Grey">
+  <material name="Grey">
     <color rgba="0.75294 0.75294 0.75294 1"/>
   </material>
   <material name="White">
     <color rgba="1 1 1 1"/>
-  </material> -->
+  </material>
 </robot>

File: pal_pro_gripper_description/urdf/pro_gripper.urdf.xacro (robot description, xacro)
@@ -38,5 +38,5 @@
       <parent link="${name}_base_link" />
       <child link="${name}_inner_finger_${side}_link" />
-      <axis xyz="0 0 -1" />
+      <axis xyz="0 0 1" />
       <limit lower="0" upper="0.81" velocity="2" effort="0.1" />
       <mimic joint="${name}_finger_joint" multiplier="1" offset="0" />
@@ -78,6 +78,6 @@
       <parent link="${name}_base_link" />
       <child link="${name}_outer_finger_${side}_link" />
-      <axis xyz="0 0 -1" />
-      <limit lower="0" upper="0.6" velocity="2" effort="0.1" />
+      <axis xyz="0 0 1" />
+      <limit lower="0" upper="${50 * deg_to_rad}" velocity="2" effort="0.1" />
       <xacro:if value="${side == 'left'}">
             <dynamics damping="0.03"/>
@@ -121,5 +121,5 @@
       <parent link="${name}_inner_finger_${side}_link" />
       <child link="${name}_fingertip_${side}_link" />
-      <axis xyz="0 0 -1" />
+      <axis xyz="0 0 1" />
       <limit lower="-0.8757" upper="0" velocity="2" effort="0.1" />
       <mimic joint="${name}_finger_joint" multiplier="-1" offset="0" />
@@ -164,6 +164,6 @@
       <provideFeedback>1</provideFeedback>
     </gazebo>
-    <xacro:pro_finger name="${name}" side="left" reflect="1" />
-    <xacro:pro_finger name="${name}" side="right" reflect="-1" />
+    <xacro:pro_finger name="${name}" side="left" reflect="-1" />
+    <xacro:pro_finger name="${name}" side="right" reflect="1" />
     <!-- Transmission only set to left outer finger joint, other joints are passive and mimic this
     joint-->
