Commit message: gripper transmission file modified

File: pal_pro_gripper_description/urdf/pro_gripper.transmission.xacro (robot description, xacro)
@@ -14,9 +14,9 @@
 <robot xmlns:xacro="http://ros.org/wiki/xacro">
   <xacro:macro name="pal_pro_gripper_transmission" params="name">
-    <transmission name="${name}_finger_trans">
+    <transmission name="${name}_trans">
         <plugin>transmission_interface/SimpleTransmission</plugin>
         <actuator name="${name}_actuator" role="actuator1"/>
-        <joint name="${name}_finger_joint" role="joint1">
-            <mechanicalReduction>1</mechanicalReduction>
+        <joint name="${name}_joint" role="joint1">
+            <mechanical_reduction>1</mechanical_reduction>
         </joint>
     </transmission>
