Commit message: Slight refactor of mimic joint ros2 control

File: pal_pro_gripper_description/urdf/pal_pro_gripper.ros2_control.xacro (robot description, xacro)
@@ -14,4 +14,14 @@
 <robot xmlns:xacro="http://ros.org/wiki/xacro">
   <xacro:macro name="ros2_control_pal_pro_gripper" params="name reduction" >
+    <xacro:macro name="ros2_control_pal_pro_gripper_mimic_joint" params="mimic_joint_name actuated_joint_name multiplier" >
+      <joint name="${mimic_joint_name}">
+        <param name="mimic">${actuated_joint_name}</param>
+        <param name="multiplier">${multiplier}</param>
+        <command_interface name="position" />
+        <state_interface name="position" />
+        <state_interface name="velocity" />
+        <state_interface name="effort" />
+      </joint>
+    </xacro:macro>
     <joint name="${name}_finger_joint">
       <command_interface name="position"/>
@@ -22,44 +32,19 @@
       <state_interface name="effort"/>
     </joint>
-    <joint name="${name}_outer_finger_right_joint">
-      <param name="mimic">${name}_finger_joint</param>
-      <param name="multiplier">1</param>
-      <command_interface name="position" />
-      <state_interface name="position" />
-      <state_interface name="velocity" />
-      <state_interface name="effort" />
-    </joint>
-    <joint name="${name}_inner_finger_left_joint">
-      <param name="mimic">${name}_finger_joint</param>
-      <param name="multiplier">1</param>
-      <command_interface name="position" />
-      <state_interface name="position" />
-      <state_interface name="velocity" />
-      <state_interface name="effort" />
-    </joint>
-    <joint name="${name}_inner_finger_right_joint">
-      <param name="mimic">${name}_finger_joint</param>
-      <param name="multiplier">1</param>
-      <command_interface name="position" />
-      <state_interface name="position" />
-      <state_interface name="velocity" />
-      <state_interface name="effort" />
-    </joint>
-    <joint name="${name}_fingertip_right_joint">
-      <param name="mimic">${name}_finger_joint</param>
-      <param name="multiplier">-1</param>
-      <command_interface name="position" />
-      <state_interface name="position" />
-      <state_interface name="velocity" />
-      <state_interface name="effort" />
-    </joint>
-    <joint name="${name}_fingertip_left_joint">
-      <param name="mimic">${name}_finger_joint</param>
-      <param name="multiplier">-1</param>
-      <command_interface name="position" />
-      <state_interface name="position" />
-      <state_interface name="velocity" />
-      <state_interface name="effort" />
-    </joint>
+    <xacro:ros2_control_pal_pro_gripper_mimic_joint mimic_joint_name="${name}_outer_finger_right_joint"
+                                                    actuated_joint_name="${name}_finger_joint"
+                                                    multiplier="1"/>
+    <xacro:ros2_control_pal_pro_gripper_mimic_joint mimic_joint_name="${name}_inner_finger_right_joint"
+                                                    actuated_joint_name="${name}_finger_joint"
+                                                    multiplier="1"/>
+    <xacro:ros2_control_pal_pro_gripper_mimic_joint mimic_joint_name="${name}_fingertip_right_joint"
+                                                    actuated_joint_name="${name}_finger_joint"
+                                                    multiplier="-1"/>
+    <xacro:ros2_control_pal_pro_gripper_mimic_joint mimic_joint_name="${name}_inner_finger_left_joint"
+                                                    actuated_joint_name="${name}_finger_joint"
+                                                    multiplier="1"/>
+    <xacro:ros2_control_pal_pro_gripper_mimic_joint mimic_joint_name="${name}_fingertip_left_joint"
+                                                    actuated_joint_name="${name}_finger_joint"
+                                                    multiplier="-1"/>
     <!-- Transmission only set to left finger joint, other joints are passive and mimic this
     joint-->
