Commit message: first commit adding description and urdf

File: pal_pro_gripper_description/urdf/pro_gripper.urdf.xacro (robot description, xacro)
@@ -47,5 +47,5 @@
     <link name="${name}_outer_finger_${side}_link">
       <inertial>
-        <origin xyz="-0.001283 0.014397 -0.000" rpy="0 0 0" />
+        <origin xyz="-0.001283 0.014397 0" rpy="0 0 0" />
         <mass value="0.015989" />
         <inertia

Commit message: update joint limits

File: pal_pro_gripper_description/urdf/pro_gripper.urdf.xacro (robot description, xacro)
@@ -38,5 +38,5 @@
       <child link="${name}_inner_finger_${side}_link" />
       <axis xyz="0 0 1" />
-      <limit lower="0" upper="0.81" velocity="2" effort="0.1" />
+      <limit lower="0" upper="${51 * deg_to_rad}" velocity="2" effort="0.1" />
       <mimic joint="${name}_finger_joint" multiplier="1" offset="0" />
     </joint>
@@ -78,5 +78,5 @@
       <child link="${name}_outer_finger_${side}_link" />
       <axis xyz="0 0 1" />
-      <limit lower="0" upper="${50 * deg_to_rad}" velocity="2" effort="0.1" />
+      <limit lower="0" upper="${51 * deg_to_rad}" velocity="2" effort="0.1" />
       <xacro:if value="${side == 'left'}">
             <dynamics damping="0.03"/>
@@ -121,5 +121,5 @@
       <child link="${name}_fingertip_${side}_link" />
       <axis xyz="0 0 1" />
-      <limit lower="-0.8757" upper="0" velocity="2" effort="0.1" />
+      <limit lower="${-51 * deg_to_rad}" upper="0" velocity="2" effort="0.1" />
       <mimic joint="${name}_finger_joint" multiplier="-1" offset="0" />
     </joint>

Commit message: Update joint limit after confirming with mechanics

File: pal_pro_gripper_description/urdf/pro_gripper.urdf.xacro (robot description, xacro)
@@ -38,5 +38,5 @@
       <child link="${name}_inner_finger_${side}_link" />
       <axis xyz="0 0 1" />
-      <limit lower="0" upper="${51 * deg_to_rad}" velocity="2" effort="0.1" />
+      <limit lower="0" upper="${53 * deg_to_rad}" velocity="2" effort="0.1" />
       <mimic joint="${name}_finger_joint" multiplier="1" offset="0" />
     </joint>
@@ -78,5 +78,5 @@
       <child link="${name}_outer_finger_${side}_link" />
       <axis xyz="0 0 1" />
-      <limit lower="0" upper="${51 * deg_to_rad}" velocity="2" effort="0.1" />
+      <limit lower="0" upper="${53 * deg_to_rad}" velocity="2" effort="0.1" />
       <xacro:if value="${side == 'left'}">
             <dynamics damping="0.03"/>
@@ -121,5 +121,5 @@
       <child link="${name}_fingertip_${side}_link" />
       <axis xyz="0 0 1" />
-      <limit lower="${-51 * deg_to_rad}" upper="0" velocity="2" effort="0.1" />
+      <limit lower="${-53 * deg_to_rad}" upper="0" velocity="2" effort="0.1" />
       <mimic joint="${name}_finger_joint" multiplier="-1" offset="0" />
     </joint>

Commit message: Add dummy link for the mimic joints

File: pal_pro_gripper_description/urdf/pro_gripper.urdf.xacro (robot description, xacro)
@@ -107,4 +107,20 @@
     </joint>
   </xacro:macro>
+    <!--Dummy joint/link to prevent error with mimic joint
+    See https://github.com/ros-controls/gazebo_ros2_control/issues/173
+    -->
+  <xacro:macro name="dummy_mimic_joint" params="name parent">
+    <link name="${name}_dummy_mimic_link"/>
+    <joint name="${name}_joint_mimic" type="fixed">
+      <parent link="${parent}" />
+      <child link="${name}_dummy_mimic_link" />
+    </joint>
+  </xacro:macro>
+  <xacro:macro name="finger_mimic_dummy" params="name side">
+    <xacro:dummy_mimic_joint name="${name}_fingertip_${side}" parent="${name}_base_link"/>
+    <xacro:dummy_mimic_joint name="${name}_inner_finger_${side}" parent="${name}_base_link"/>
+    <!-- <xacro:dummy_mimic_joint name="${prefix}${fingerprefix}_outer_finger_right_joint" parent="${prefix}base_link"/> -->
+    <!-- <xacro:dummy_mimic_joint name="${prefix}${fingerprefix}_inner_knuckle" parent="${prefix}base_link"/> -->
+  </xacro:macro>
   <xacro:macro name="pal_pro_gripper" params="name parent *origin">
     <link name="${name}_base_link">
@@ -178,4 +194,8 @@
     <xacro:pro_finger name="${name}" side="left" reflect="-1" />
     <xacro:pro_finger name="${name}" side="right" reflect="1" />
+    <!-- Temporary fix until mimic joint works properly with MoveIt!-->
+    <xacro:finger_mimic_dummy name="${name}" side="right"/>
+    <xacro:finger_mimic_dummy name="${name}" side="left"/>
+    <xacro:dummy_mimic_joint name="${name}_outer_finger_right" parent="${name}_base_link"/>
   </xacro:macro>
 </robot>

Commit message: Update gripper joint limit based on new encoder reduction of 81

File: pal_pro_gripper_description/urdf/pro_gripper.urdf.xacro (robot description, xacro)
@@ -31,5 +31,5 @@
       <child link="${name}_inner_finger_${side}_link" />
       <axis xyz="0 0 1" />
-      <limit lower="0" upper="${53 * deg_to_rad}" velocity="2" effort="0.1" />
+      <limit lower="0" upper="${46 * deg_to_rad}" velocity="2" effort="0.1" />
       <mimic joint="${name}_finger_joint" multiplier="1" offset="0" />
     </joint>
@@ -67,5 +67,5 @@
       <child link="${name}_outer_finger_${side}_link" />
       <axis xyz="0 0 1" />
-      <limit lower="0" upper="${53 * deg_to_rad}" velocity="2" effort="0.1" />
+      <limit lower="0" upper="${46 * deg_to_rad}" velocity="2" effort="0.1" />
       <xacro:if value="${side == 'left'}">
             <dynamics damping="0.03"/>
@@ -103,5 +103,5 @@
       <child link="${name}_fingertip_${side}_link" />
       <axis xyz="0 0 1" />
-      <limit lower="${-53 * deg_to_rad}" upper="0" velocity="2" effort="0.1" />
+      <limit lower="${-46 * deg_to_rad}" upper="0" velocity="2" effort="0.1" />
       <mimic joint="${name}_finger_joint" multiplier="-1" offset="0" />
     </joint>
