Commit message: Proper base origin and offset

File: pal_pro_gripper_description/urdf/gripper.properties.xacro (robot description, xacro)
@@ -24,6 +24,6 @@
         </inertial>
     </xacro:macro>
-    <xacro:macro name="origin_inner_finger_joint" params="reflect">
-        <origin xyz="0 ${reflect * 0.013977} 0.078832" rpy="1.5708 0.83776 ${reflect * 1.5708}" />
+    <xacro:macro name="origin_inner_finger_joint" params="reflect offset">
+        <origin xyz="0 ${reflect * 0.013977} ${0.078832 + offset}" rpy="1.5708 0.83776 ${reflect * 1.5708}" />
     </xacro:macro>
     <!-- Outer finger -->
@@ -35,6 +35,6 @@
         </inertial>
     </xacro:macro>
-    <xacro:macro name="origin_outer_finger_joint" params="reflect">
-        <origin xyz="0 ${reflect * 0.0288} 0.0743" rpy="1.5708 0.83776 ${reflect * 1.5708}" />
+    <xacro:macro name="origin_outer_finger_joint" params="reflect offset">
+        <origin xyz="0 ${reflect * 0.0288} ${0.0743 + offset}" rpy="1.5708 0.83776 ${reflect * 1.5708}" />
     </xacro:macro>
     <!-- Fingertip -->

File: pal_pro_gripper_description/urdf/gripper.urdf.xacro (robot description, xacro)
@@ -2,5 +2,5 @@
 <robot xmlns:xacro="http://ros.org/wiki/xacro">
   <!-- A finger of the pal_pro_gripper -->
-  <xacro:macro name="pro_finger" params="name side reflect">
+  <xacro:macro name="pro_finger" params="name side reflect finger_offset:=0">
     <!-- Inner finger -->
     <link name="${name}_inner_finger_${side}_link">
@@ -23,5 +23,5 @@
     </link>
     <joint name="${name}_inner_finger_${side}_joint" type="revolute">
-      <xacro:origin_inner_finger_joint reflect="${reflect}" />
+      <xacro:origin_inner_finger_joint reflect="${reflect}" offset="${finger_offset}"/>
       <parent link="${name}_base_link" />
       <child link="${name}_inner_finger_${side}_link" />
@@ -52,5 +52,5 @@
     <xacro:property name="outer_finger_joint_name" value="${name + '_finger_joint' if side == 'left' else name + '_outer_finger_' + side + '_joint'}" />
     <joint name="${outer_finger_joint_name}" type="revolute">
-      <xacro:origin_outer_finger_joint reflect="${reflect}"/>
+      <xacro:origin_outer_finger_joint reflect="${reflect}" offset="${finger_offset}"/>
       <parent link="${name}_base_link" />
       <child link="${name}_outer_finger_${side}_link" />
@@ -93,7 +93,8 @@
   </xacro:macro>
   <!-- GRIPPER DEFINITION -->
-  <xacro:macro name="pal_pro_gripper" params="tool_changer name parent *origin">
+  <xacro:macro name="pal_pro_gripper" params="tool_changer:=False name parent *origin">
     <!-- Vesion name depending if it is a prototype -->
     <xacro:property name="base_type" value="${'base_link_tc' if tool_changer else 'base_link_ntc'}" />
+    <xacro:property name="finger_offset" value="${0.0 if tool_changer else 0.006}" />
     <!-- Properties files -->
     <xacro:include filename="$(find pal_pro_gripper_description)/urdf/gripper.properties.xacro"/>
@@ -127,6 +128,6 @@
     </joint>
     <!-- Fingers -->
-    <xacro:pro_finger name="${name}" side="left" reflect="-1" />
-    <xacro:pro_finger name="${name}" side="right" reflect="1" />
+    <xacro:pro_finger name="${name}" side="left" reflect="-1" finger_offset="${finger_offset}"/>
+    <xacro:pro_finger name="${name}" side="right" reflect="1" finger_offset="${finger_offset}"/>
     <!-- Gazebo config -->
     <gazebo reference="${name}_inner_finger_left_link">

Commit message: Update griper base link Inertias

File: pal_pro_gripper_description/urdf/gripper.properties.xacro (robot description, xacro)
@@ -3,7 +3,7 @@
     <xacro:macro name="inertial_base_link_tc">
         <inertial>
-            <origin xyz="-0.000111195944040731 -5.20000467719152E-05 0.04682714296137" rpy="0 0 0" />
-            <mass value="0.351833020899102" />
-            <inertia ixx="0.000212702588837237" ixy="-1.5724450163606E-07" ixz="4.66935789777261E-07" iyy="0.000159938323491697" iyz="-1.90446642900145E-07" izz="0.000254149142086845" />
+            <origin xyz="-5.081E-05 6.06E-06 0.04330857" rpy="0 0 0" />
+            <mass value="0.59671873" />
+            <inertia ixx="0.00064209" ixy="-2.1E-07" ixz="6.5E-07" iyy="0.00060742" iyz="2.1E-07" izz="0.00037836" />
         </inertial>
     </xacro:macro>

Commit message: Fixing urdf and ros2control

File: pal_pro_gripper_description/urdf/gripper.properties.xacro (robot description, xacro)
@@ -25,5 +25,5 @@
     </xacro:macro>
     <xacro:macro name="origin_inner_finger_joint" params="reflect offset">
-        <origin xyz="0 ${reflect * 0.013977} ${0.078832 + offset}" rpy="1.5708 0.83776 ${reflect * 1.5708}" />
+        <origin xyz="-0.01482273272 0.00453176142 0.0" rpy="0.0 0.0 0.0" />
     </xacro:macro>
     <!-- Outer finger -->
@@ -49,3 +49,25 @@
         <origin xyz="0 0.05 0" rpy="0 0 0" />
     </xacro:macro>
+    <!-- Screw -->
+    <xacro:macro name="inertial_screw_link">
+        <inertial>
+            <origin xyz="0.0 0.0 0.0" rpy="0 0 0" />
+            <mass value="0.02" />
+            <inertia ixx="7.4666667e-07" ixy="0.0" ixz="0.0" iyy="7.4666667e-07" iyz="0.0" izz="1.6e-07" />
+        </inertial>
+    </xacro:macro>
+    <xacro:macro name="origin_screw_joint" params="reflect">
+        <origin xyz="-0.0178 0.0088 0.0" rpy="0 0 0"/>
+    </xacro:macro>
+    <!-- Base finger -->
+    <xacro:macro name="inertial_base_finger_link">
+        <inertial>
+            <origin xyz="0.0 0.0 0.0" rpy="0 0 0" />
+            <mass value="0.02" />
+            <inertia ixx="7.4666667e-07" ixy="0.0" ixz="0.0" iyy="7.4666667e-07" iyz="0.0" izz="1.6e-07" />
+        </inertial>
+    </xacro:macro>
+    <xacro:macro name="origin_base_finger_joint" params="reflect">
+    <origin xyz="0.0 ${reflect * 0.0288} 0.07565" rpy="1.5708 0 ${reflect * 1.5708}"/>
+    </xacro:macro>
 </robot>

File: pal_pro_gripper_description/urdf/gripper.ros2_control.xacro (robot description, xacro)
@@ -20,5 +20,5 @@
       </joint>
     </xacro:macro>
-    <joint name="${name}_finger_joint">
+    <joint name="${name}_screw_joint">
       <command_interface name="position"/>
       <state_interface name="position">
@@ -28,14 +28,15 @@
       <state_interface name="effort"/>
     </joint>
-    <xacro:ros2_control_pal_pro_gripper_mimic_joint mimic_joint_name="${name}_outer_finger_right_joint" actuated_joint_name="${name}_finger_joint" multiplier="1"/>
-    <xacro:ros2_control_pal_pro_gripper_mimic_joint mimic_joint_name="${name}_inner_finger_right_joint" actuated_joint_name="${name}_finger_joint" multiplier="1"/>
-    <xacro:ros2_control_pal_pro_gripper_mimic_joint mimic_joint_name="${name}_fingertip_right_joint" actuated_joint_name="${name}_finger_joint" multiplier="-1"/>
-    <xacro:ros2_control_pal_pro_gripper_mimic_joint mimic_joint_name="${name}_inner_finger_left_joint" actuated_joint_name="${name}_finger_joint" multiplier="1"/>
-    <xacro:ros2_control_pal_pro_gripper_mimic_joint mimic_joint_name="${name}_fingertip_left_joint" actuated_joint_name="${name}_finger_joint" multiplier="-1"/>
+    <xacro:ros2_control_pal_pro_gripper_mimic_joint mimic_joint_name="${name}_outer_finger_right_joint" actuated_joint_name="${name}_screw_joint" multiplier="-37.281"/>
+    <xacro:ros2_control_pal_pro_gripper_mimic_joint mimic_joint_name="${name}_inner_finger_right_joint" actuated_joint_name="${name}_screw_joint" multiplier="-37.281"/>
+    <xacro:ros2_control_pal_pro_gripper_mimic_joint mimic_joint_name="${name}_fingertip_right_joint" actuated_joint_name="${name}_screw_joint" multiplier="37.281"/>
+    <xacro:ros2_control_pal_pro_gripper_mimic_joint mimic_joint_name="${name}_outer_finger_left_joint" actuated_joint_name="${name}_screw_joint" multiplier="-37.281"/>
+    <xacro:ros2_control_pal_pro_gripper_mimic_joint mimic_joint_name="${name}_inner_finger_left_joint" actuated_joint_name="${name}_screw_joint" multiplier="-37.281"/>
+    <xacro:ros2_control_pal_pro_gripper_mimic_joint mimic_joint_name="${name}_fingertip_left_joint" actuated_joint_name="${name}_screw_joint" multiplier="37.281"/>
     <!-- Transmission only set to left finger joint, other joints are passive and mimic this
     joint-->
     <xacro:if value="${sim_type not in ['mujoco', 'mujoco-ros2-control']}">
       <xacro:include filename="$(find pal_pro_gripper_description)/urdf/gripper.transmission.xacro" />
-      <xacro:pal_pro_gripper_transmission name="${name}_finger"/>
+      <xacro:pal_pro_gripper_transmission name="${name}_screw"/>
     </xacro:if>
   </xacro:macro>

File: pal_pro_gripper_description/urdf/gripper.transmission.xacro (robot description, xacro)
@@ -15,9 +15,13 @@
   <xacro:macro name="pal_pro_gripper_transmission" params="name">
     <transmission name="${name}_trans">
-        <plugin>transmission_interface/SimpleTransmission</plugin>
+        <!-- <plugin>transmission_interface/SimpleTransmission</plugin> -->
+        <plugin>pal_pro_gripper_transmissions/PalGripperTransmission</plugin>
         <actuator name="${name}_actuator" role="actuator1"/>
         <joint name="${name}_joint" role="joint1">
-            <mechanical_reduction>1</mechanical_reduction>
+            <!-- <mechanical_reduction>1</mechanical_reduction> -->
+            <mechanical_reduction>81</mechanical_reduction>
         </joint>
+        <!-- Needs to be used in the real robot -->
+        <!-- <param name="func_type">d2l</param>   -->
     </transmission>
   </xacro:macro>

File: pal_pro_gripper_description/urdf/gripper.urdf.xacro (robot description, xacro)
@@ -3,20 +3,77 @@
   <!-- A finger of the pal_pro_gripper -->
   <xacro:macro name="pro_finger" params="name side reflect finger_offset:=0">
+    <!-- Screw link -->
+    <link name="${name}_screw_${side}_link">
+      <xacro:inertial_screw_link />
+      <visual>
+        <origin xyz="0 0 0" rpy="0 0 0"/>
+        <geometry>
+          <sphere radius="0.004"/>
+        </geometry>
+        <material name="">
+          <color rgba="0.752941176470588 0.752941176470588 0.752941176470588 1" />
+        </material>
+      </visual>
+      <collision>
+        <origin xyz="0 0 0" rpy="0 0 0"/>
+        <geometry>
+          <sphere radius="0.004"/>
+        </geometry>
+      </collision>
+    </link>
+    <xacro:property name="screw_joint_name" value="${name + '_screw_joint' if side == 'left' else name + '_screw_' + side + '_joint'}" />
+    <joint name="${screw_joint_name}" type="prismatic">
+      <xacro:origin_screw_joint reflect="${reflect}"/>
+      <parent link="${name}_base_finger_${side}_link"/>
+      <child link="${name}_screw_${side}_link"/>
+      <axis xyz="0 1 0"/>
+      <limit lower="0.001327" upper="0.017638" velocity="2" effort="0.1"/>
+       <xacro:if value="${side == 'left'}">
+        <dynamics damping="0.03"/>
+      </xacro:if>
+      <xacro:unless value="${side == 'left'}">
+        <mimic joint="${name}_screw_joint" multiplier="1" offset="0" />
+      </xacro:unless>
+    </joint>
+    <!-- Gripper base finger link-->
+    <link name='${name}_base_finger_${side}_link'>
+      <xacro:inertial_base_finger_link/>
+      <visual>
+        <origin xyz="0 0 0" rpy="0 0 0"/>
+        <geometry>
+          <sphere radius="0.005"/>
+        </geometry>
+        <material name="">
+          <color rgba="0.752941176470588 0.752941176470588 0.752941176470588 1" />
+        </material>
+      </visual>
+      <collision>
+        <origin xyz="0 0 0" rpy="0 0 0"/>
+        <geometry>
+          <sphere radius="0.005"/>
+        </geometry>
+      </collision>
+    </link>
+    <joint name="${name}_base_finger_${side}_joint" type="fixed">
+      <xacro:origin_base_finger_joint reflect="${reflect}"/>
+      <parent link="${name}_base_link"/>
+      <child link="${name}_base_finger_${side}_link"/>
+    </joint>
     <!-- Inner finger -->
     <link name="${name}_inner_finger_${side}_link">
       <xacro:inertial_inner_finger_link />
       <visual>
-        <origin xyz="0 0 0" rpy="0 0 0" />
-        <geometry>
-          <mesh filename="package://pal_pro_gripper_description/meshes/inner_finger.stl" />
-        </geometry>
-        <material name="">
-          <color rgba="0.752941176470588 0.752941176470588 0.752941176470588 1" />
-        </material>
-      </visual>
-      <collision>
-        <origin xyz="0 0 0" rpy="0 0 0" />
-        <geometry>
-          <mesh filename="package://pal_pro_gripper_description/meshes/inner_finger.stl" />
+        <origin xyz="0 0 0" rpy="0 0 0"/>
+        <geometry>
+          <mesh filename="package://pal_pro_gripper_description/meshes/inner_finger.stl"/>
+        </geometry>
+        <material name="">
+          <color rgba="0.752941176470588 0.752941176470588 0.752941176470588 1" />
+        </material>
+      </visual>
+      <collision>
+        <origin xyz="0 0 0" rpy="0 0 0"/>
+        <geometry>
+          <mesh filename="package://pal_pro_gripper_description/meshes/inner_finger.stl"/>
         </geometry>
       </collision>
@@ -24,9 +81,9 @@
     <joint name="${name}_inner_finger_${side}_joint" type="revolute">
       <xacro:origin_inner_finger_joint reflect="${reflect}" offset="${finger_offset}"/>
-      <parent link="${name}_base_link" />
-      <child link="${name}_inner_finger_${side}_link" />
-      <axis xyz="0 0 -1" />
-      <limit lower="${-46 * deg_to_rad}" upper="0" velocity="2" effort="0.1"/>
-      <mimic joint="${name}_finger_joint" multiplier="1" offset="${-46 * deg_to_rad}" />
+      <parent link="${name}_base_finger_${side}_link"/>
+      <child link="${name}_inner_finger_${side}_link"/>
+      <axis xyz="0 0 1"/>
+      <limit lower="${59.548 * deg_to_rad}" upper="${107.619 * deg_to_rad}" velocity="2" effort="0.1"/>
+      <mimic joint="${name}_screw_joint" multiplier="-37.281" offset="0.0"/>
     </joint>
     <!-- Outer finger -->
@@ -34,33 +91,26 @@
       <xacro:inertial_outer_finger_link />
       <visual>
-        <origin xyz="0 0 0" rpy="0 0 0" />
-        <geometry>
-          <mesh filename="package://pal_pro_gripper_description/meshes/outer_finger.stl" />
-        </geometry>
-        <material name="">
-          <color rgba="0.752941176470588 0.752941176470588 0.752941176470588 1" />
-        </material>
-      </visual>
-      <collision>
-        <origin xyz="0 0 0" rpy="0 0 0" />
-        <geometry>
-          <mesh filename="package://pal_pro_gripper_description/meshes/outer_finger.stl" />
-        </geometry>
-      </collision>
-    </link>
-    <!--  The left outer joint is set as gripper_finger_joint. All other joints are passive and will mimic this joint-->
-    <xacro:property name="outer_finger_joint_name" value="${name + '_finger_joint' if side == 'left' else name + '_outer_finger_' + side + '_joint'}" />
-    <joint name="${outer_finger_joint_name}" type="revolute">
+        <origin xyz="0 0 0" rpy="0 0 0"/>
+        <geometry>
+          <mesh filename="package://pal_pro_gripper_description/meshes/outer_finger.stl"/>
+        </geometry>
+        <material name="">
+          <color rgba="0.752941176470588 0.752941176470588 0.752941176470588 1" />
+        </material>
+      </visual>
+      <collision>
+        <origin xyz="0 0 0" rpy="0 0 0"/>
+        <geometry>
+          <mesh filename="package://pal_pro_gripper_description/meshes/outer_finger.stl"/>
+        </geometry>
+      </collision>
+    </link>
+    <joint name="${name}_outer_finger_${side}_joint" type="revolute">
       <xacro:origin_outer_finger_joint reflect="${reflect}" offset="${finger_offset}"/>
-      <parent link="${name}_base_link" />
-      <child link="${name}_outer_finger_${side}_link" />
-      <axis xyz="0 0 -1" />
-      <limit lower="0.0" upper="${46 * deg_to_rad}" velocity="2" effort="0.1" />
-      <xacro:if value="${side == 'left'}">
-        <dynamics damping="0.03"/>
-      </xacro:if>
-      <xacro:unless value="${side == 'left'}">
-        <mimic joint="${name}_finger_joint" multiplier="1" offset="0.0" />
-      </xacro:unless>
+      <parent link="${name}_base_link"/>
+      <child link="${name}_outer_finger_${side}_link"/>
+      <axis xyz="0 0 1"/>
+      <limit lower="${41.999 * deg_to_rad}" upper="${92.838 * deg_to_rad}" velocity="2" effort="0.1"/>
+      <mimic joint="${name}_screw_joint" multiplier="-37.281" offset="0.0"/>
     </joint>
     <!-- Fingertip -->
@@ -68,26 +118,26 @@
       <xacro:inertial_fingertip_link />
       <visual>
-        <origin xyz="0 0 0" rpy="0 0 0" />
-        <geometry>
-          <mesh filename="package://pal_pro_gripper_description/meshes/fingertip.stl" />
-        </geometry>
-        <material name="">
-          <color rgba="0.752941176470588 0.752941176470588 0.752941176470588 1" />
-        </material>
-      </visual>
-      <collision>
-        <origin xyz="0 0 0" rpy="0 0 0" />
-        <geometry>
-          <mesh filename="package://pal_pro_gripper_description/meshes/fingertip.stl" />
+        <origin xyz="0 0 0" rpy="0 0 0"/>
+        <geometry>
+          <mesh filename="package://pal_pro_gripper_description/meshes/fingertip.stl"/>
+        </geometry>
+        <material name="">
+          <color rgba="0.752941176470588 0.752941176470588 0.752941176470588 1" />
+        </material>
+      </visual>
+      <collision>
+        <origin xyz="0 0 0" rpy="0 0 0"/>
+        <geometry>
+          <mesh filename="package://pal_pro_gripper_description/meshes/fingertip.stl"/>
         </geometry>
       </collision>
     </link>
     <joint name="${name}_fingertip_${side}_joint" type="revolute">
-      <xacro:origin_fingertip_joint reflect="${reflect}" />
-      <parent link="${name}_inner_finger_${side}_link" />
-      <child link="${name}_fingertip_${side}_link" />
-      <axis xyz="0 0 -1" />
-      <limit lower="${-46 * deg_to_rad}" upper="0" velocity="2" effort="0.1"/>
-      <mimic joint="${name}_finger_joint" multiplier="-1" offset="0" />
+      <xacro:origin_fingertip_joint reflect="${reflect}"/>
+      <parent link="${name}_inner_finger_${side}_link"/>
+      <child link="${name}_fingertip_${side}_link"/>
+      <axis xyz="0 0 1"/>
+      <limit lower="${59.548 * deg_to_rad}" upper="${107.619 * deg_to_rad}" velocity="2" effort="0.1"/>
+      <mimic joint="${name}_screw_joint" multiplier="37.281" offset="0.0"/>
     </joint>
   </xacro:macro>
@@ -178,11 +228,25 @@
       <mu2>0.9</mu2>
     </gazebo>
-    <gazebo reference="${name}_finger_joint">
-      <implicitSpringDamper>1</implicitSpringDamper>
-      <provideFeedback>1</provideFeedback>
-    </gazebo>
-    <gazebo reference="${name}_finger_joint">
-      <implicitSpringDamper>1</implicitSpringDamper>
-      <provideFeedback>1</provideFeedback>
+    <!-- Screw links -->
+    <gazebo reference="${name}_screw_joint">
+      <material>Gazebo/DarkGrey</material>
+      <mu1>0.9</mu1>
+      <mu2>0.9</mu2>
+    </gazebo>
+    <gazebo reference="${name}_screw_joint">
+      <material>Gazebo/DarkGrey</material>
+      <mu1>0.9</mu1>
+      <mu2>0.9</mu2>
+    </gazebo>
+    <!-- Base finger links -->
+    <gazebo reference="${name}_base_finger_left_link">
+      <material>Gazebo/DarkGrey</material>
+      <mu1>0.9</mu1>
+      <mu2>0.9</mu2>
+    </gazebo>
+    <gazebo reference="${name}_base_finger_right_link">
+      <material>Gazebo/DarkGrey</material>
+      <mu1>0.9</mu1>
+      <mu2>0.9</mu2>
     </gazebo>
   </xacro:macro>
