Commit message: changing limits joints

File: pal_pro_gripper_description/urdf/gripper.properties.xacro (robot description, xacro)
@@ -57,5 +57,5 @@
         </inertial>
     </xacro:macro>
-    <xacro:macro name="origin_screw_joint" params="reflect">
+    <xacro:macro name="origin_finger_joint" params="reflect">
         <origin xyz="-0.0178 0.0088 0.0" rpy="0 0 0"/>
     </xacro:macro>

File: pal_pro_gripper_description/urdf/gripper.ros2_control.xacro (robot description, xacro)
@@ -20,5 +20,5 @@
       </joint>
     </xacro:macro>
-    <joint name="${name}_screw_joint">
+    <joint name="${name}_finger_joint">
       <command_interface name="position"/>
       <state_interface name="position">
@@ -32,20 +32,19 @@
       <state_interface name="effort"/>
     </joint>
-    <xacro:ros2_control_pal_pro_gripper_mimic_joint mimic_joint_name="${name}_outer_finger_right_joint" actuated_joint_name="${name}_screw_joint" multiplier="-37.281"/>
-    <xacro:ros2_control_pal_pro_gripper_mimic_joint mimic_joint_name="${name}_inner_finger_right_joint" actuated_joint_name="${name}_screw_joint" multiplier="-37.281"/>
-    <xacro:ros2_control_pal_pro_gripper_mimic_joint mimic_joint_name="${name}_fingertip_right_joint" actuated_joint_name="${name}_screw_joint" multiplier="37.281"/>
-<<<<<<< HEAD
+    <xacro:ros2_control_pal_pro_gripper_mimic_joint mimic_joint_name="${name}_outer_finger_right_joint" actuated_joint_name="${name}_finger_joint" multiplier="-37.281"/>
+    <xacro:ros2_control_pal_pro_gripper_mimic_joint mimic_joint_name="${name}_inner_finger_right_joint" actuated_joint_name="${name}_finger_joint" multiplier="-37.281"/>
+    <xacro:ros2_control_pal_pro_gripper_mimic_joint mimic_joint_name="${name}_fingertip_right_joint" actuated_joint_name="${name}_finger_joint" multiplier="37.281"/>
     <xacro:ros2_control_pal_pro_gripper_mimic_joint mimic_joint_name="${name}_screw_right_joint" actuated_joint_name="${name}_screw_joint" multiplier="1.0"/>
+    <xacro:ros2_control_pal_pro_gripper_mimic_joint mimic_joint_name="${name}_screw_right_joint" actuated_joint_name="${name}_finger_joint" multiplier="1.0"/>
+    <xacro:ros2_control_pal_pro_gripper_mimic_joint mimic_joint_name="${name}_outer_finger_left_joint" actuated_joint_name="${name}_finger_joint" multiplier="-37.281"/>
     <xacro:ros2_control_pal_pro_gripper_mimic_joint mimic_joint_name="${name}_outer_finger_left_joint" actuated_joint_name="${name}_screw_joint" multiplier="-37.281"/>
-=======
-    <xacro:ros2_control_pal_pro_gripper_mimic_joint mimic_joint_name="${name}_outer_finger_left_joint" actuated_joint_name="${name}_screw_joint" multiplier="-37.281"/>
->>>>>>> b225891 (fixing rebase)
     <xacro:ros2_control_pal_pro_gripper_mimic_joint mimic_joint_name="${name}_inner_finger_left_joint" actuated_joint_name="${name}_screw_joint" multiplier="-37.281"/>
-    <xacro:ros2_control_pal_pro_gripper_mimic_joint mimic_joint_name="${name}_fingertip_left_joint" actuated_joint_name="${name}_screw_joint" multiplier="37.281"/>
+    <xacro:ros2_control_pal_pro_gripper_mimic_joint mimic_joint_name="${name}_inner_finger_left_joint" actuated_joint_name="${name}_finger_joint" multiplier="-37.281"/>
+    <xacro:ros2_control_pal_pro_gripper_mimic_joint mimic_joint_name="${name}_fingertip_left_joint" actuated_joint_name="${name}_finger_joint" multiplier="37.281"/>
     <!-- Transmission only set to left finger joint, other joints are passive and mimic this
     joint-->
     <xacro:if value="${sim_type not in ['mujoco', 'mujoco-ros2-control']}">
       <xacro:include filename="$(find pal_pro_gripper_description)/urdf/gripper.transmission.xacro" />
-      <xacro:pal_pro_gripper_transmission name="${name}_screw"/>
+      <xacro:pal_pro_gripper_transmission name="${name}_finger"/>
     </xacro:if>
   </xacro:macro>

File: pal_pro_gripper_description/urdf/gripper.transmission.xacro (robot description, xacro)
@@ -15,6 +15,6 @@
   <xacro:macro name="pal_pro_gripper_transmission" params="name">
     <transmission name="${name}_trans">
-        <!-- <plugin>transmission_interface/SimpleTransmission</plugin> -->
-        <plugin>pal_pro_gripper_transmissions/PalGripperTransmission</plugin>
+        <plugin>transmission_interface/SimpleTransmission</plugin>
+        <!-- <plugin>pal_pro_gripper_transmissions/PalGripperTransmission</plugin> -->
         <actuator name="${name}_actuator" role="actuator1"/>
         <joint name="${name}_joint" role="joint1">

File: pal_pro_gripper_description/urdf/gripper.urdf.xacro (robot description, xacro)
@@ -22,7 +22,7 @@
       </collision>
     </link>
-    <xacro:property name="screw_joint_name" value="${name + '_screw_joint' if side == 'left' else name + '_screw_' + side + '_joint'}" />
-    <joint name="${screw_joint_name}" type="prismatic">
-      <xacro:origin_screw_joint reflect="${reflect}"/>
+    <xacro:property name="finger_joint_name" value="${name + '_finger_joint' if side == 'left' else name + '_screw_' + side + '_joint'}" />
+    <joint name="${finger_joint_name}" type="prismatic">
+      <xacro:origin_finger_joint reflect="${reflect}"/>
       <parent link="${name}_base_finger_${side}_link"/>
       <child link="${name}_screw_${side}_link"/>
@@ -33,5 +33,5 @@
       </xacro:if>
       <xacro:unless value="${side == 'left'}">
-        <mimic joint="${name}_screw_joint" multiplier="1" offset="0" />
+        <mimic joint="${name}_finger_joint" multiplier="1" offset="0" />
       </xacro:unless>
     </joint>
@@ -85,5 +85,5 @@
       <axis xyz="0 0 1"/>
       <limit lower="${-42.840* deg_to_rad}" upper="${8.001 * deg_to_rad}" velocity="2" effort="0.1"/>
-      <mimic joint="${name}_screw_joint" multiplier="-37.281" offset="0.0"/>
+      <mimic joint="${name}_finger_joint" multiplier="-37.281" offset="0.0"/>
     </joint>
     <!-- Outer finger -->
@@ -112,5 +112,5 @@
       <axis xyz="0 0 1"/>
       <limit lower="${-42.840 * deg_to_rad}" upper="${8.001 * deg_to_rad}" velocity="2" effort="0.1"/>
-      <mimic joint="${name}_screw_joint" multiplier="-37.281" offset="0.0"/>
+      <mimic joint="${name}_finger_joint" multiplier="-37.281" offset="0.0"/>
     </joint>
     <!-- Fingertip -->
@@ -139,5 +139,5 @@
       <axis xyz="0 0 1"/>
       <limit lower="${-8.001 * deg_to_rad}" upper="${42.840 * deg_to_rad}" velocity="2" effort="0.1"/>
-      <mimic joint="${name}_screw_joint" multiplier="37.281" offset="0.0"/>
+      <mimic joint="${name}_finger_joint" multiplier="37.281" offset="0.0"/>
     </joint>
   </xacro:macro>
@@ -229,10 +229,10 @@
     </gazebo>
     <!-- Screw links -->
-    <gazebo reference="${name}_screw_joint">
-      <material>Gazebo/DarkGrey</material>
-      <mu1>0.9</mu1>
-      <mu2>0.9</mu2>
-    </gazebo>
-    <gazebo reference="${name}_screw_joint">
+    <gazebo reference="${name}_finger_joint">
+      <material>Gazebo/DarkGrey</material>
+      <mu1>0.9</mu1>
+      <mu2>0.9</mu2>
+    </gazebo>
+    <gazebo reference="${name}_finger_joint">
       <material>Gazebo/DarkGrey</material>
       <mu1>0.9</mu1>

Commit message: fix range gripper urdf

File: pal_pro_gripper_description/urdf/gripper.properties.xacro (robot description, xacro)
@@ -36,5 +36,5 @@
     </xacro:macro>
     <xacro:macro name="origin_outer_finger_joint" params="reflect offset">
-        <origin xyz="0 ${reflect * 0.0288} ${0.0743 + offset}" rpy="1.5708 0.83776 ${reflect * 1.5708}" />
+        <origin xyz="0.0 ${reflect * 0.0288} 0.07565" rpy="1.5708 0 ${reflect * 1.5708}"/>
     </xacro:macro>
     <!-- Fingertip -->
@@ -47,5 +47,5 @@
     </xacro:macro>
     <xacro:macro name="origin_fingertip_joint" params="reflect">
-        <origin xyz="0 0.05 0" rpy="0 0 0.83776" />
+        <origin xyz="0 0.05 0" rpy="0 0 0" />
     </xacro:macro>
 </robot>

File: pal_pro_gripper_description/urdf/gripper.ros2_control.xacro (robot description, xacro)
@@ -23,5 +23,5 @@
       <command_interface name="position"/>
       <state_interface name="position">
-        <param name="initial_value">0.15</param>
+        <param name="initial_value">0.0</param>
       </state_interface>
       <state_interface name="velocity"/>
@@ -31,5 +31,5 @@
     <xacro:ros2_control_pal_pro_gripper_mimic_joint mimic_joint_name="${name}_inner_finger_right_joint" actuated_joint_name="${name}_finger_joint" multiplier="1"/>
     <xacro:ros2_control_pal_pro_gripper_mimic_joint mimic_joint_name="${name}_fingertip_right_joint" actuated_joint_name="${name}_finger_joint" multiplier="-1"/>
-    <xacro:ros2_control_pal_pro_gripper_mimic_joint mimic_joint_name="${name}_inner_finger_left_joint" actuated_joint_name="${name}_finger_joint" multiplier="1"/>
+    <xacro:ros2_control_pal_pro_gripper_mimic_joint mimic_joint_name="${name}_inner_finger_left_joint" actuated_joint_name="${name}_finger_joint" multiplier="1}"/>
     <xacro:ros2_control_pal_pro_gripper_mimic_joint mimic_joint_name="${name}_fingertip_left_joint" actuated_joint_name="${name}_finger_joint" multiplier="-1"/>
     <!-- Transmission only set to left finger joint, other joints are passive and mimic this

File: pal_pro_gripper_description/urdf/gripper.urdf.xacro (robot description, xacro)
@@ -26,11 +26,11 @@
       <parent link="${name}_base_link" />
       <child link="${name}_inner_finger_${side}_link" />
-      <axis xyz="0 0 1" />
-      <limit lower="0" upper="${46 * deg_to_rad}" velocity="2" effort="0.1" />
-      <mimic joint="${name}_finger_joint" multiplier="1" offset="0" />
+      <axis xyz="0 0 -1" />
+      <limit lower="${-46 * deg_to_rad}" upper="0" velocity="2" effort="0.1"/>
+      <mimic joint="${name}_finger_joint" multiplier="1" offset="${-46 * deg_to_rad}" />
     </joint>
     <!-- Outer finger -->
     <link name="${name}_outer_finger_${side}_link">
-      <xacro:inertial_outer_finger_link />
+      <xacro:inertial_outer_finger_link/>
       <visual>
         <origin xyz="0 0 0" rpy="0 0 0" />
@@ -55,11 +55,11 @@
       <parent link="${name}_base_link" />
       <child link="${name}_outer_finger_${side}_link" />
-      <axis xyz="0 0 1" />
-      <limit lower="0" upper="${54.431 * deg_to_rad}" velocity="2" effort="0.1" />
+      <axis xyz="0 0 -1" />
+      <limit lower="0.0" upper="${46 * deg_to_rad}" velocity="2" effort="0.1" />
       <xacro:if value="${side == 'left'}">
         <dynamics damping="0.03"/>
       </xacro:if>
       <xacro:unless value="${side == 'left'}">
-        <mimic joint="${name}_finger_joint" multiplier="1" offset="0" />
+        <mimic joint="${name}_finger_joint" multiplier="1" offset="0.0" />
       </xacro:unless>
     </joint>
@@ -87,6 +87,6 @@
       <parent link="${name}_inner_finger_${side}_link" />
       <child link="${name}_fingertip_${side}_link" />
-      <axis xyz="0 0 1" />
-      <limit lower="${-46 * deg_to_rad}" upper="0" velocity="2" effort="0.1" />
+      <axis xyz="0 0 -1" />
+      <limit lower="${-46 * deg_to_rad}" upper="0" velocity="2" effort="0.1"/>
       <mimic joint="${name}_finger_joint" multiplier="-1" offset="0" />
     </joint>
