Commit message: Update range of gripper

File: pal_pro_gripper_description/urdf/gripper.urdf.xacro (robot description, xacro)
@@ -56,5 +56,5 @@
       <child link="${name}_outer_finger_${side}_link" />
       <axis xyz="0 0 1" />
-      <limit lower="0" upper="${46 * deg_to_rad}" velocity="2" effort="0.1" />
+      <limit lower="0" upper="${54.431 * deg_to_rad}" velocity="2" effort="0.1" />
       <xacro:if value="${side == 'left'}">
         <dynamics damping="0.03"/>

Commit message: Changing revolute joint limits

File: pal_pro_gripper_description/urdf/gripper.urdf.xacro (robot description, xacro)
@@ -84,5 +84,5 @@
       <child link="${name}_inner_finger_${side}_link"/>
       <axis xyz="0 0 1"/>
-      <limit lower="${59.548 * deg_to_rad}" upper="${107.619 * deg_to_rad}" velocity="2" effort="0.1"/>
+      <limit lower="0" upper="${53 * deg_to_rad}" velocity="2" effort="0.1"/>
       <mimic joint="${name}_screw_joint" multiplier="-37.281" offset="0.0"/>
     </joint>
@@ -111,5 +111,5 @@
       <child link="${name}_outer_finger_${side}_link"/>
       <axis xyz="0 0 1"/>
-      <limit lower="${41.999 * deg_to_rad}" upper="${92.838 * deg_to_rad}" velocity="2" effort="0.1"/>
+      <limit lower="0" upper="${53 * deg_to_rad}" velocity="2" effort="0.1"/>
       <mimic joint="${name}_screw_joint" multiplier="-37.281" offset="0.0"/>
     </joint>
@@ -138,5 +138,5 @@
       <child link="${name}_fingertip_${side}_link"/>
       <axis xyz="0 0 1"/>
-      <limit lower="${59.548 * deg_to_rad}" upper="${107.619 * deg_to_rad}" velocity="2" effort="0.1"/>
+      <limit lower="${-53 * deg_to_rad}" upper="0" velocity="2" effort="0.1"/>
       <mimic joint="${name}_screw_joint" multiplier="37.281" offset="0.0"/>
     </joint>

Commit message: adding use_sim_time

File: pal_pro_gripper_description/urdf/gripper.urdf.xacro (robot description, xacro)
@@ -3,4 +3,5 @@
   <!-- A finger of the pal_pro_gripper -->
   <xacro:macro name="pro_finger" params="name side reflect finger_offset:=0">
+  <xacro:arg name="use_sim_time" default="false"/>
     <!-- Screw link -->
     <link name="${name}_screw_${side}_link">
@@ -28,9 +29,11 @@
       <child link="${name}_screw_${side}_link"/>
       <axis xyz="0 1 0"/>
-      <!-- Use this limits for simulation-->
-      <!-- <limit lower="0.001327" upper="0.017638" velocity="2" effort="0.1"/> -->
-      <!-- Use this limits for real robot-->
-      <limit lower="0.0" upper="0.07938" velocity="2" effort="0.1"/>
-       <xacro:if value="${side == 'left'}">
+      <xacro:if value="$(arg use_sim_time)">
+        <limit lower="0.001327" upper="0.017638" velocity="2" effort="0.1"/>
+      </xacro:if>
+      <xacro:unless value="$(arg use_sim_time)">
+        <limit lower="0.0" upper="0.07938" velocity="2" effort="0.1"/>
+      </xacro:unless>
+      <xacro:if value="${side == 'left'}">
         <dynamics damping="0.03"/>
       </xacro:if>
