Commit message: Gripper std and suggested changes

File: pal_pro_gripper_description/urdf/gripper.ros2_control.xacro (robot description, xacro)
@@ -11,5 +11,5 @@
 See the License for the specific language governing permissions and
 limitations under the License.
- -->
+-->
 <robot xmlns:xacro="http://ros.org/wiki/xacro">
   <xacro:macro name="ros2_control_pal_pro_gripper" params="name reduction">

File: pal_pro_gripper_description/urdf/gripper.urdf.xacro (robot description, xacro)
@@ -95,5 +95,5 @@
   <xacro:macro name="pal_pro_gripper" params="tool_changer:=False name parent *origin">
     <!-- Vesion name depending if it is a prototype -->
-    <xacro:property name="base_type" value="${'base_link_tc' if tool_changer else 'base_link_ntc'}" />
+    <xacro:property name="gripper_base_type" value="${'base_link_tc' if tool_changer else 'base_link_ntc'}" />
     <xacro:property name="finger_offset" value="${0.0 if tool_changer else 0.006}" />
     <!-- Properties files -->
@@ -110,5 +110,5 @@
         <origin xyz="0 0 0" rpy="0 0 0" />
         <geometry>
-          <mesh filename="package://pal_pro_gripper_description/meshes/${base_type}.stl" />
+          <mesh filename="package://pal_pro_gripper_description/meshes/${gripper_base_type}.stl" />
         </geometry>
         <material name="pal/DarkGrey" />
@@ -117,5 +117,5 @@
         <origin xyz="0 0 0" rpy="0 0 0" />
         <geometry>
-          <mesh filename="package://pal_pro_gripper_description/meshes/${base_type}.stl" />
+          <mesh filename="package://pal_pro_gripper_description/meshes/${gripper_base_type}.stl" />
         </geometry>
       </collision>

Commit message: Fixing urdf and ros2control

File: pal_pro_gripper_description/urdf/gripper.ros2_control.xacro (robot description, xacro)
@@ -20,5 +20,5 @@
       </joint>
     </xacro:macro>
-    <joint name="${name}_finger_joint">
+    <joint name="${name}_screw_joint">
       <command_interface name="position"/>
       <state_interface name="position">
@@ -43,5 +43,5 @@
     <xacro:if value="${sim_type not in ['mujoco', 'mujoco-ros2-control']}">
       <xacro:include filename="$(find pal_pro_gripper_description)/urdf/gripper.transmission.xacro" />
-      <xacro:pal_pro_gripper_transmission name="${name}_finger"/>
+      <xacro:pal_pro_gripper_transmission name="${name}_screw"/>
     </xacro:if>
   </xacro:macro>

File: pal_pro_gripper_description/urdf/gripper.transmission.xacro (robot description, xacro)
@@ -15,6 +15,11 @@
   <xacro:macro name="pal_pro_gripper_transmission" params="name">
     <transmission name="${name}_trans">
+<<<<<<< HEAD
         <plugin>transmission_interface/SimpleTransmission</plugin>
         <!-- <plugin>pal_pro_gripper_transmissions/PalGripperTransmission</plugin> -->
+=======
+        <!-- <plugin>transmission_interface/SimpleTransmission</plugin> -->
+        <plugin>pal_pro_gripper_transmissions/PalGripperTransmission</plugin>
+>>>>>>> d4c60e9 (Fixing urdf and ros2control)
         <actuator name="${name}_actuator" role="actuator1"/>
         <joint name="${name}_joint" role="joint1">

Commit message: Fixing limits joint

File: pal_pro_gripper_description/urdf/gripper.ros2_control.xacro (robot description, xacro)
@@ -23,5 +23,9 @@
       <command_interface name="position"/>
       <state_interface name="position">
+<<<<<<< HEAD
         <param name="initial_value">0.0</param>
+=======
+        <param name="initial_value">0.002</param>
+>>>>>>> 8b271f0 (Fixing limits joint)
       </state_interface>
       <state_interface name="velocity"/>
@@ -31,4 +35,5 @@
     <xacro:ros2_control_pal_pro_gripper_mimic_joint mimic_joint_name="${name}_inner_finger_right_joint" actuated_joint_name="${name}_screw_joint" multiplier="-37.281"/>
     <xacro:ros2_control_pal_pro_gripper_mimic_joint mimic_joint_name="${name}_fingertip_right_joint" actuated_joint_name="${name}_screw_joint" multiplier="37.281"/>
+    <xacro:ros2_control_pal_pro_gripper_mimic_joint mimic_joint_name="${name}_screw_right_joint" actuated_joint_name="${name}_screw_joint" multiplier="1.0"/>
     <xacro:ros2_control_pal_pro_gripper_mimic_joint mimic_joint_name="${name}_outer_finger_left_joint" actuated_joint_name="${name}_screw_joint" multiplier="-37.281"/>
     <xacro:ros2_control_pal_pro_gripper_mimic_joint mimic_joint_name="${name}_inner_finger_left_joint" actuated_joint_name="${name}_screw_joint" multiplier="-37.281"/>

File: pal_pro_gripper_description/urdf/gripper.urdf.xacro (robot description, xacro)
@@ -9,14 +9,14 @@
         <origin xyz="0 0 0" rpy="0 0 0"/>
         <geometry>
-          <sphere radius="0.004"/>
-        </geometry>
-        <material name="">
-          <color rgba="0.752941176470588 0.752941176470588 0.752941176470588 1" />
-        </material>
-      </visual>
-      <collision>
-        <origin xyz="0 0 0" rpy="0 0 0"/>
-        <geometry>
-          <sphere radius="0.004"/>
+          <sphere radius="0.002"/>
+        </geometry>
+        <material name="">
+          <color rgba="0.752941176470588 0.752941176470588 0.752941176470588 1" />
+        </material>
+      </visual>
+      <collision>
+        <origin xyz="0 0 0" rpy="0 0 0"/>
+        <geometry>
+          <sphere radius="0.002"/>
         </geometry>
       </collision>
@@ -42,14 +42,14 @@
         <origin xyz="0 0 0" rpy="0 0 0"/>
         <geometry>
-          <sphere radius="0.005"/>
-        </geometry>
-        <material name="">
-          <color rgba="0.752941176470588 0.752941176470588 0.752941176470588 1" />
-        </material>
-      </visual>
-      <collision>
-        <origin xyz="0 0 0" rpy="0 0 0"/>
-        <geometry>
-          <sphere radius="0.005"/>
+          <sphere radius="0.001"/>
+        </geometry>
+        <material name="">
+          <color rgba="0.752941176470588 0.752941176470588 0.752941176470588 1" />
+        </material>
+      </visual>
+      <collision>
+        <origin xyz="0 0 0" rpy="0 0 0"/>
+        <geometry>
+          <sphere radius="0.001"/>
         </geometry>
       </collision>
@@ -84,5 +84,5 @@
       <child link="${name}_inner_finger_${side}_link"/>
       <axis xyz="0 0 1"/>
-      <limit lower="0" upper="${53 * deg_to_rad}" velocity="2" effort="0.1"/>
+      <limit lower="${-42.840* deg_to_rad}" upper="${8.001 * deg_to_rad}" velocity="2" effort="0.1"/>
       <mimic joint="${name}_screw_joint" multiplier="-37.281" offset="0.0"/>
     </joint>
@@ -111,5 +111,5 @@
       <child link="${name}_outer_finger_${side}_link"/>
       <axis xyz="0 0 1"/>
-      <limit lower="0" upper="${53 * deg_to_rad}" velocity="2" effort="0.1"/>
+      <limit lower="${-42.840 * deg_to_rad}" upper="${8.001 * deg_to_rad}" velocity="2" effort="0.1"/>
       <mimic joint="${name}_screw_joint" multiplier="-37.281" offset="0.0"/>
     </joint>
@@ -138,5 +138,5 @@
       <child link="${name}_fingertip_${side}_link"/>
       <axis xyz="0 0 1"/>
-      <limit lower="${-53 * deg_to_rad}" upper="0" velocity="2" effort="0.1"/>
+      <limit lower="${-8.001 * deg_to_rad}" upper="${42.840 * deg_to_rad}" velocity="2" effort="0.1"/>
       <mimic joint="${name}_screw_joint" multiplier="37.281" offset="0.0"/>
     </joint>
@@ -250,4 +250,12 @@
       <mu2>0.9</mu2>
     </gazebo>
+    <gazebo>
+      <plugin name="mimic_joint_plugin_right" filename="libgazebo_ros_mimic_joint.so">
+        <joint>gripper_screw_left_joint</joint>
+        <mimicJoint>gripper_screw_right_joint</mimicJoint>
+        <multiplier>1.0</multiplier>
+        <offset>0.0</offset>
+      </plugin>
+    </gazebo>
   </xacro:macro>
 </robot>

Commit message: fix

File: pal_pro_gripper_description/urdf/gripper.ros2_control.xacro (robot description, xacro)
@@ -35,6 +35,10 @@
     <xacro:ros2_control_pal_pro_gripper_mimic_joint mimic_joint_name="${name}_inner_finger_right_joint" actuated_joint_name="${name}_screw_joint" multiplier="-37.281"/>
     <xacro:ros2_control_pal_pro_gripper_mimic_joint mimic_joint_name="${name}_fingertip_right_joint" actuated_joint_name="${name}_screw_joint" multiplier="37.281"/>
+<<<<<<< HEAD
     <xacro:ros2_control_pal_pro_gripper_mimic_joint mimic_joint_name="${name}_screw_right_joint" actuated_joint_name="${name}_screw_joint" multiplier="1.0"/>
     <xacro:ros2_control_pal_pro_gripper_mimic_joint mimic_joint_name="${name}_outer_finger_left_joint" actuated_joint_name="${name}_screw_joint" multiplier="-37.281"/>
+=======
+    <xacro:ros2_control_pal_pro_gripper_mimic_joint mimic_joint_name="${name}_outer_finger_left_joint" actuated_joint_name="${name}_screw_joint" multiplier="-37.281"/>
+>>>>>>> b225891 (fixing rebase)
     <xacro:ros2_control_pal_pro_gripper_mimic_joint mimic_joint_name="${name}_inner_finger_left_joint" actuated_joint_name="${name}_screw_joint" multiplier="-37.281"/>
     <xacro:ros2_control_pal_pro_gripper_mimic_joint mimic_joint_name="${name}_fingertip_left_joint" actuated_joint_name="${name}_screw_joint" multiplier="37.281"/>

File: pal_pro_gripper_description/urdf/gripper.urdf.xacro (robot description, xacro)
@@ -258,4 +258,15 @@
       </plugin>
     </gazebo>
+    <!-- Base finger links -->
+    <gazebo reference="${name}_base_finger_left_link">
+      <material>Gazebo/DarkGrey</material>
+      <mu1>0.9</mu1>
+      <mu2>0.9</mu2>
+    </gazebo>
+    <gazebo reference="${name}_base_finger_right_link">
+      <material>Gazebo/DarkGrey</material>
+      <mu1>0.9</mu1>
+      <mu2>0.9</mu2>
+    </gazebo>
   </xacro:macro>
 </robot>

Commit message: fix xacro

File: pal_pro_gripper_description/urdf/gripper.ros2_control.xacro (robot description, xacro)
@@ -20,5 +20,5 @@
       </joint>
     </xacro:macro>
-    <joint name="${name}_screw_joint">
+    <joint name="${name}_finger_joint">
       <command_interface name="position"/>
       <state_interface name="position">
@@ -35,5 +35,5 @@
     <xacro:ros2_control_pal_pro_gripper_mimic_joint mimic_joint_name="${name}_inner_finger_right_joint" actuated_joint_name="${name}_finger_joint" multiplier="-37.281"/>
     <xacro:ros2_control_pal_pro_gripper_mimic_joint mimic_joint_name="${name}_fingertip_right_joint" actuated_joint_name="${name}_finger_joint" multiplier="37.281"/>
-    <xacro:ros2_control_pal_pro_gripper_mimic_joint mimic_joint_name="${name}_screw_right_joint" actuated_joint_name="${name}_finger_joint" multiplier="1.0"/>
+    <xacro:ros2_control_pal_pro_gripper_mimic_joint mimic_joint_name="${name}_finger_right_joint" actuated_joint_name="${name}_finger_joint" multiplier="1.0"/>
     <xacro:ros2_control_pal_pro_gripper_mimic_joint mimic_joint_name="${name}_outer_finger_left_joint" actuated_joint_name="${name}_finger_joint" multiplier="-37.281"/>
     <xacro:ros2_control_pal_pro_gripper_mimic_joint mimic_joint_name="${name}_inner_finger_left_joint" actuated_joint_name="${name}_finger_joint" multiplier="-37.281"/>
@@ -43,5 +43,5 @@
     <xacro:if value="${sim_type not in ['mujoco', 'mujoco-ros2-control']}">
       <xacro:include filename="$(find pal_pro_gripper_description)/urdf/gripper.transmission.xacro" />
-      <xacro:pal_pro_gripper_transmission name="${name}_screw"/>
+      <xacro:pal_pro_gripper_transmission name="${name}_finger"/>
     </xacro:if>
   </xacro:macro>

File: pal_pro_gripper_description/urdf/gripper.transmission.xacro (robot description, xacro)
@@ -15,6 +15,6 @@
   <xacro:macro name="pal_pro_gripper_transmission" params="name">
     <transmission name="${name}_trans">
-        <plugin>transmission_interface/SimpleTransmission</plugin>
-        <!-- <plugin>pal_pro_gripper_transmissions/PalGripperTransmission</plugin> -->
+        <!-- <plugin>transmission_interface/SimpleTransmission</plugin> -->
+        <plugin>pal_pro_gripper_transmissions/PalGripperTransmission</plugin>
         <actuator name="${name}_actuator" role="actuator1"/>
         <joint name="${name}_joint" role="joint1">

File: pal_pro_gripper_description/urdf/gripper.urdf.xacro (robot description, xacro)
@@ -22,5 +22,5 @@
       </collision>
     </link>
-    <xacro:property name="finger_joint_name" value="${name + '_finger_joint' if side == 'left' else name + '_screw_' + side + '_joint'}" />
+    <xacro:property name="finger_joint_name" value="${name + '_finger_joint' if side == 'left' else name + '_finger_' + side + '_joint'}" />
     <joint name="${finger_joint_name}" type="prismatic">
       <xacro:origin_finger_joint reflect="${reflect}"/>
@@ -252,6 +252,6 @@
     <gazebo>
       <plugin name="mimic_joint_plugin_right" filename="libgazebo_ros_mimic_joint.so">
-        <joint>gripper_screw_left_joint</joint>
-        <mimicJoint>gripper_screw_right_joint</mimicJoint>
+        <joint>gripper_finger_joint</joint>
+        <mimicJoint>gripper_finger_right_joint</mimicJoint>
         <multiplier>1.0</multiplier>
         <offset>0.0</offset>

Commit message: changes ros2control

File: pal_pro_gripper_description/urdf/gripper.ros2_control.xacro (robot description, xacro)
@@ -20,28 +20,24 @@
       </joint>
     </xacro:macro>
-    <joint name="${name}_finger_joint">
+    <joint name="${name}_screw_joint">
       <command_interface name="position"/>
       <state_interface name="position">
-<<<<<<< HEAD
-        <param name="initial_value">0.0</param>
-=======
         <param name="initial_value">0.002</param>
->>>>>>> 8b271f0 (Fixing limits joint)
       </state_interface>
       <state_interface name="velocity"/>
       <state_interface name="effort"/>
     </joint>
-    <xacro:ros2_control_pal_pro_gripper_mimic_joint mimic_joint_name="${name}_outer_finger_right_joint" actuated_joint_name="${name}_finger_joint" multiplier="-37.281"/>
-    <xacro:ros2_control_pal_pro_gripper_mimic_joint mimic_joint_name="${name}_inner_finger_right_joint" actuated_joint_name="${name}_finger_joint" multiplier="-37.281"/>
-    <xacro:ros2_control_pal_pro_gripper_mimic_joint mimic_joint_name="${name}_fingertip_right_joint" actuated_joint_name="${name}_finger_joint" multiplier="37.281"/>
-    <xacro:ros2_control_pal_pro_gripper_mimic_joint mimic_joint_name="${name}_finger_right_joint" actuated_joint_name="${name}_finger_joint" multiplier="1.0"/>
-    <xacro:ros2_control_pal_pro_gripper_mimic_joint mimic_joint_name="${name}_outer_finger_left_joint" actuated_joint_name="${name}_finger_joint" multiplier="-37.281"/>
-    <xacro:ros2_control_pal_pro_gripper_mimic_joint mimic_joint_name="${name}_inner_finger_left_joint" actuated_joint_name="${name}_finger_joint" multiplier="-37.281"/>
-    <xacro:ros2_control_pal_pro_gripper_mimic_joint mimic_joint_name="${name}_fingertip_left_joint" actuated_joint_name="${name}_finger_joint" multiplier="37.281"/>
+    <xacro:ros2_control_pal_pro_gripper_mimic_joint mimic_joint_name="${name}_outer_finger_right_joint" actuated_joint_name="${name}_screw_joint" multiplier="-37.281"/>
+    <xacro:ros2_control_pal_pro_gripper_mimic_joint mimic_joint_name="${name}_inner_finger_right_joint" actuated_joint_name="${name}_screw_joint" multiplier="-37.281"/>
+    <xacro:ros2_control_pal_pro_gripper_mimic_joint mimic_joint_name="${name}_fingertip_right_joint" actuated_joint_name="${name}_screw_joint" multiplier="37.281"/>
+    <xacro:ros2_control_pal_pro_gripper_mimic_joint mimic_joint_name="${name}_screw_right_joint" actuated_joint_name="${name}_screw_joint" multiplier="1.0"/>
+    <xacro:ros2_control_pal_pro_gripper_mimic_joint mimic_joint_name="${name}_outer_finger_left_joint" actuated_joint_name="${name}_screw_joint" multiplier="-37.281"/>
+    <xacro:ros2_control_pal_pro_gripper_mimic_joint mimic_joint_name="${name}_inner_finger_left_joint" actuated_joint_name="${name}_screw_joint" multiplier="-37.281"/>
+    <xacro:ros2_control_pal_pro_gripper_mimic_joint mimic_joint_name="${name}_fingertip_left_joint" actuated_joint_name="${name}_screw_joint" multiplier="37.281"/>
     <!-- Transmission only set to left finger joint, other joints are passive and mimic this
     joint-->
     <xacro:if value="${sim_type not in ['mujoco', 'mujoco-ros2-control']}">
       <xacro:include filename="$(find pal_pro_gripper_description)/urdf/gripper.transmission.xacro" />
-      <xacro:pal_pro_gripper_transmission name="${name}_finger"/>
+      <xacro:pal_pro_gripper_transmission name="${name}_screw"/>
     </xacro:if>
   </xacro:macro>

Commit message: fixing values gripper

File: pal_pro_gripper_description/urdf/gripper.ros2_control.xacro (robot description, xacro)
@@ -23,5 +23,5 @@
       <command_interface name="position"/>
       <state_interface name="position">
-        <param name="initial_value">0.002</param>
+        <param name="initial_value">0.039</param>
       </state_interface>
       <state_interface name="velocity"/>

File: pal_pro_gripper_description/urdf/gripper.transmission.xacro (robot description, xacro)
@@ -19,6 +19,5 @@
         <actuator name="${name}_actuator" role="actuator1"/>
         <joint name="${name}_joint" role="joint1">
-            <!-- <mechanical_reduction>1</mechanical_reduction> -->
-            <mechanical_reduction>81</mechanical_reduction>
+            <mechanical_reduction>1.0</mechanical_reduction>
         </joint>
         <!-- Needs to be used in the real robot -->

File: pal_pro_gripper_description/urdf/gripper.urdf.xacro (robot description, xacro)
@@ -28,5 +28,8 @@
       <child link="${name}_screw_${side}_link"/>
       <axis xyz="0 1 0"/>
-      <limit lower="0.001327" upper="0.017638" velocity="2" effort="0.1"/>
+      <!-- Use this limits for simulation-->
+      <!-- <limit lower="0.001327" upper="0.017638" velocity="2" effort="0.1"/> -->
+      <!-- Use this limits for real robot-->
+      <limit lower="0.0" upper="0.07938" velocity="2" effort="0.1"/>
        <xacro:if value="${side == 'left'}">
         <dynamics damping="0.03"/>

Commit message: fix ros2control

File: pal_pro_gripper_description/urdf/gripper.ros2_control.xacro (robot description, xacro)
@@ -20,5 +20,5 @@
       </joint>
     </xacro:macro>
-    <joint name="${name}_screw_joint">
+    <joint name="${name}_finger_joint">
       <command_interface name="position"/>
       <state_interface name="position">
@@ -28,16 +28,16 @@
       <state_interface name="effort"/>
     </joint>
-    <xacro:ros2_control_pal_pro_gripper_mimic_joint mimic_joint_name="${name}_outer_finger_right_joint" actuated_joint_name="${name}_screw_joint" multiplier="-37.281"/>
-    <xacro:ros2_control_pal_pro_gripper_mimic_joint mimic_joint_name="${name}_inner_finger_right_joint" actuated_joint_name="${name}_screw_joint" multiplier="-37.281"/>
-    <xacro:ros2_control_pal_pro_gripper_mimic_joint mimic_joint_name="${name}_fingertip_right_joint" actuated_joint_name="${name}_screw_joint" multiplier="37.281"/>
-    <xacro:ros2_control_pal_pro_gripper_mimic_joint mimic_joint_name="${name}_screw_right_joint" actuated_joint_name="${name}_screw_joint" multiplier="1.0"/>
-    <xacro:ros2_control_pal_pro_gripper_mimic_joint mimic_joint_name="${name}_outer_finger_left_joint" actuated_joint_name="${name}_screw_joint" multiplier="-37.281"/>
-    <xacro:ros2_control_pal_pro_gripper_mimic_joint mimic_joint_name="${name}_inner_finger_left_joint" actuated_joint_name="${name}_screw_joint" multiplier="-37.281"/>
-    <xacro:ros2_control_pal_pro_gripper_mimic_joint mimic_joint_name="${name}_fingertip_left_joint" actuated_joint_name="${name}_screw_joint" multiplier="37.281"/>
+    <xacro:ros2_control_pal_pro_gripper_mimic_joint mimic_joint_name="${name}_outer_finger_right_joint" actuated_joint_name="${name}_finger_joint" multiplier="-37.281"/>
+    <xacro:ros2_control_pal_pro_gripper_mimic_joint mimic_joint_name="${name}_inner_finger_right_joint" actuated_joint_name="${name}_finger_joint" multiplier="-37.281"/>
+    <xacro:ros2_control_pal_pro_gripper_mimic_joint mimic_joint_name="${name}_fingertip_right_joint" actuated_joint_name="${name}_finger_joint" multiplier="37.281"/>
+    <xacro:ros2_control_pal_pro_gripper_mimic_joint mimic_joint_name="${name}_finger_right_joint" actuated_joint_name="${name}_finger_joint" multiplier="1.0"/>
+    <xacro:ros2_control_pal_pro_gripper_mimic_joint mimic_joint_name="${name}_outer_finger_left_joint" actuated_joint_name="${name}_finger_joint" multiplier="-37.281"/>
+    <xacro:ros2_control_pal_pro_gripper_mimic_joint mimic_joint_name="${name}_inner_finger_left_joint" actuated_joint_name="${name}_finger_joint" multiplier="-37.281"/>
+    <xacro:ros2_control_pal_pro_gripper_mimic_joint mimic_joint_name="${name}_fingertip_left_joint" actuated_joint_name="${name}_finger_joint" multiplier="37.281"/>
     <!-- Transmission only set to left finger joint, other joints are passive and mimic this
     joint-->
     <xacro:if value="${sim_type not in ['mujoco', 'mujoco-ros2-control']}">
       <xacro:include filename="$(find pal_pro_gripper_description)/urdf/gripper.transmission.xacro" />
-      <xacro:pal_pro_gripper_transmission name="${name}_screw"/>
+      <xacro:pal_pro_gripper_transmission name="${name}_finger"/>
     </xacro:if>
   </xacro:macro>
