Commit message: fixing urdf gripper

File: pal_pro_gripper_description/urdf/gripper.ros2_control.xacro (robot description, xacro)
@@ -28,11 +28,11 @@
       <state_interface name="effort"/>
     </joint>
-    <xacro:ros2_control_pal_pro_gripper_mimic_joint mimic_joint_name="${name}_outer_finger_right_joint" actuated_joint_name="${name}_finger_joint" multiplier="-37.281"/>
-    <xacro:ros2_control_pal_pro_gripper_mimic_joint mimic_joint_name="${name}_inner_finger_right_joint" actuated_joint_name="${name}_finger_joint" multiplier="-37.281"/>
-    <xacro:ros2_control_pal_pro_gripper_mimic_joint mimic_joint_name="${name}_fingertip_right_joint" actuated_joint_name="${name}_finger_joint" multiplier="37.281"/>
-    <xacro:ros2_control_pal_pro_gripper_mimic_joint mimic_joint_name="${name}_finger_right_joint" actuated_joint_name="${name}_finger_joint" multiplier="1.0"/>
-    <xacro:ros2_control_pal_pro_gripper_mimic_joint mimic_joint_name="${name}_outer_finger_left_joint" actuated_joint_name="${name}_finger_joint" multiplier="-37.281"/>
-    <xacro:ros2_control_pal_pro_gripper_mimic_joint mimic_joint_name="${name}_inner_finger_left_joint" actuated_joint_name="${name}_finger_joint" multiplier="-37.281"/>
-    <xacro:ros2_control_pal_pro_gripper_mimic_joint mimic_joint_name="${name}_fingertip_left_joint" actuated_joint_name="${name}_finger_joint" multiplier="37.281"/>
+    <xacro:ros2_control_pal_pro_gripper_mimic_joint mimic_joint_name="${name}_outer_finger_right_joint" actuated_joint_name="${name}_finger_joint" multiplier="-8.28"/>
+    <xacro:ros2_control_pal_pro_gripper_mimic_joint mimic_joint_name="${name}_inner_finger_right_joint" actuated_joint_name="${name}_finger_joint" multiplier="-8.28"/>
+    <xacro:ros2_control_pal_pro_gripper_mimic_joint mimic_joint_name="${name}_fingertip_right_joint" actuated_joint_name="${name}_finger_joint" multiplier="8.28"/>
+    <xacro:ros2_control_pal_pro_gripper_mimic_joint mimic_joint_name="${name}_finger_right_joint" actuated_joint_name="${name}_finger_joint" multiplier="0.22"/>
+    <xacro:ros2_control_pal_pro_gripper_mimic_joint mimic_joint_name="${name}_outer_finger_left_joint" actuated_joint_name="${name}_finger_joint" multiplier="-8.28"/>
+    <xacro:ros2_control_pal_pro_gripper_mimic_joint mimic_joint_name="${name}_inner_finger_left_joint" actuated_joint_name="${name}_finger_joint" multiplier="-8.28"/>
+    <xacro:ros2_control_pal_pro_gripper_mimic_joint mimic_joint_name="${name}_fingertip_left_joint" actuated_joint_name="${name}_finger_joint" multiplier="8.28"/>
     <!-- Transmission only set to left finger joint, other joints are passive and mimic this
     joint-->

File: pal_pro_gripper_description/urdf/gripper.urdf.xacro (robot description, xacro)
@@ -3,23 +3,7 @@
   <!-- A finger of the pal_pro_gripper -->
   <xacro:macro name="pro_finger" params="name side reflect finger_offset:=0">
-  <xacro:arg name="use_sim_time" default="false"/>
     <!-- Screw link -->
     <link name="${name}_screw_${side}_link">
       <xacro:inertial_screw_link />
-      <visual>
-        <origin xyz="0 0 0" rpy="0 0 0"/>
-        <geometry>
-          <sphere radius="0.002"/>
-        </geometry>
-        <material name="">
-          <color rgba="0.752941176470588 0.752941176470588 0.752941176470588 1" />
-        </material>
-      </visual>
-      <collision>
-        <origin xyz="0 0 0" rpy="0 0 0"/>
-        <geometry>
-          <sphere radius="0.002"/>
-        </geometry>
-      </collision>
     </link>
     <xacro:property name="finger_joint_name" value="${name + '_finger_joint' if side == 'left' else name + '_finger_' + side + '_joint'}" />
@@ -29,15 +13,10 @@
       <child link="${name}_screw_${side}_link"/>
       <axis xyz="0 1 0"/>
-      <xacro:if value="$(arg use_sim_time)">
-        <limit lower="0.001327" upper="0.017638" velocity="2" effort="0.1"/>
-      </xacro:if>
-      <xacro:unless value="$(arg use_sim_time)">
-        <limit lower="0.0" upper="0.07938" velocity="2" effort="0.1"/>
-      </xacro:unless>
+      <limit lower="0.0" upper="0.07938" velocity="2" effort="0.1"/>
       <xacro:if value="${side == 'left'}">
         <dynamics damping="0.03"/>
       </xacro:if>
       <xacro:unless value="${side == 'left'}">
-        <mimic joint="${name}_finger_joint" multiplier="1" offset="0" />
+        <mimic joint="${name}_finger_joint" multiplier="0.22" offset="0" />
       </xacro:unless>
     </joint>
@@ -91,5 +70,5 @@
       <axis xyz="0 0 1"/>
       <limit lower="${-42.840* deg_to_rad}" upper="${8.001 * deg_to_rad}" velocity="2" effort="0.1"/>
-      <mimic joint="${name}_finger_joint" multiplier="-37.281" offset="0.0"/>
+      <mimic joint="${name}_finger_joint" multiplier="-8.28" offset="0.0"/>
     </joint>
     <!-- Outer finger -->
@@ -118,5 +97,5 @@
       <axis xyz="0 0 1"/>
       <limit lower="${-42.840 * deg_to_rad}" upper="${8.001 * deg_to_rad}" velocity="2" effort="0.1"/>
-      <mimic joint="${name}_finger_joint" multiplier="-37.281" offset="0.0"/>
+      <mimic joint="${name}_finger_joint" multiplier="-8.28" offset="0.0"/>
     </joint>
     <!-- Fingertip -->
@@ -145,5 +124,5 @@
       <axis xyz="0 0 1"/>
       <limit lower="${-8.001 * deg_to_rad}" upper="${42.840 * deg_to_rad}" velocity="2" effort="0.1"/>
-      <mimic joint="${name}_finger_joint" multiplier="37.281" offset="0.0"/>
+      <mimic joint="${name}_finger_joint" multiplier="8.28" offset="0.0"/>
     </joint>
   </xacro:macro>

Commit message: try to fix gripper mimic (not working yet)

File: pal_pro_gripper_description/urdf/gripper.ros2_control.xacro (robot description, xacro)
@@ -18,4 +18,11 @@
         <param name="mimic">${actuated_joint_name}</param>
         <param name="multiplier">${multiplier}</param>
+        <!-- state_interface lets GazeboSimSystem track the physical joint position.
+             hardware_interface propagates the mimic state automatically from the
+             URDF <mimic> tag. Command is enforced in Gazebo via
+             JointPositionController plugin + gripper_mimic_relay node. -->
+        <xacro:if value="${sim_type == 'gazebo'}">
+          <state_interface name="position"/>
+        </xacro:if>
       </joint>
     </xacro:macro>
@@ -28,14 +35,14 @@
       <state_interface name="effort"/>
     </joint>
-    <xacro:ros2_control_pal_pro_gripper_mimic_joint mimic_joint_name="${name}_outer_finger_right_joint" actuated_joint_name="${name}_finger_joint" multiplier="-8.28"/>
-    <xacro:ros2_control_pal_pro_gripper_mimic_joint mimic_joint_name="${name}_inner_finger_right_joint" actuated_joint_name="${name}_finger_joint" multiplier="-8.28"/>
-    <xacro:ros2_control_pal_pro_gripper_mimic_joint mimic_joint_name="${name}_fingertip_right_joint" actuated_joint_name="${name}_finger_joint" multiplier="8.28"/>
-    <xacro:ros2_control_pal_pro_gripper_mimic_joint mimic_joint_name="${name}_finger_right_joint" actuated_joint_name="${name}_finger_joint" multiplier="0.22"/>
-    <xacro:ros2_control_pal_pro_gripper_mimic_joint mimic_joint_name="${name}_outer_finger_left_joint" actuated_joint_name="${name}_finger_joint" multiplier="-8.28"/>
-    <xacro:ros2_control_pal_pro_gripper_mimic_joint mimic_joint_name="${name}_inner_finger_left_joint" actuated_joint_name="${name}_finger_joint" multiplier="-8.28"/>
-    <xacro:ros2_control_pal_pro_gripper_mimic_joint mimic_joint_name="${name}_fingertip_left_joint" actuated_joint_name="${name}_finger_joint" multiplier="8.28"/>
+    <xacro:ros2_control_pal_pro_gripper_mimic_joint mimic_joint_name="${name}_outer_finger_right_joint" actuated_joint_name="${name}_finger_joint" multiplier="-8.28" sim_type="${sim_type}"/>
+    <xacro:ros2_control_pal_pro_gripper_mimic_joint mimic_joint_name="${name}_inner_finger_right_joint" actuated_joint_name="${name}_finger_joint" multiplier="-8.28" sim_type="${sim_type}"/>
+    <xacro:ros2_control_pal_pro_gripper_mimic_joint mimic_joint_name="${name}_fingertip_right_joint" actuated_joint_name="${name}_finger_joint" multiplier="8.28" sim_type="${sim_type}"/>
+    <xacro:ros2_control_pal_pro_gripper_mimic_joint mimic_joint_name="${name}_finger_right_joint" actuated_joint_name="${name}_finger_joint" multiplier="0.22" sim_type="${sim_type}"/>
+    <xacro:ros2_control_pal_pro_gripper_mimic_joint mimic_joint_name="${name}_outer_finger_left_joint" actuated_joint_name="${name}_finger_joint" multiplier="-8.28" sim_type="${sim_type}"/>
+    <xacro:ros2_control_pal_pro_gripper_mimic_joint mimic_joint_name="${name}_inner_finger_left_joint" actuated_joint_name="${name}_finger_joint" multiplier="-8.28" sim_type="${sim_type}"/>
+    <xacro:ros2_control_pal_pro_gripper_mimic_joint mimic_joint_name="${name}_fingertip_left_joint" actuated_joint_name="${name}_finger_joint" multiplier="8.28" sim_type="${sim_type}"/>
     <!-- Transmission only set to left finger joint, other joints are passive and mimic this
     joint-->
-    <xacro:if value="${sim_type not in ['mujoco', 'mujoco-ros2-control']}">
+    <xacro:if value="${sim_type == 'no-simulation'}">
       <xacro:include filename="$(find pal_pro_gripper_description)/urdf/gripper.transmission.xacro" />
       <xacro:pal_pro_gripper_transmission name="${name}_finger"/>

File: pal_pro_gripper_description/urdf/gripper.urdf.xacro (robot description, xacro)
@@ -213,4 +213,30 @@
     <xacro:pro_finger name="${name}" side="left" reflect="-1" finger_offset="${finger_offset}"/>
     <xacro:pro_finger name="${name}" side="right" reflect="1" finger_offset="${finger_offset}"/>
+    <!-- Gazebo mimic joint enforcement via JointPositionController.
+         sdformat_urdf drops URDF <mimic> tags so Gazebo physics does not enforce
+         the mechanical coupling. Each mimic joint gets a Gazebo PID controller
+         driven by the gripper_mimic_relay ROS2 node via ros_gz_bridge.
+         Topic convention: /gz_gripper_mimic/{joint_full_name} -->
+    <xacro:macro name="gz_mimic_joint_controller" params="joint_name">
+      <gazebo>
+        <plugin filename="gz-sim-joint-position-controller-system"
+                name="gz::sim::systems::JointPositionController">
+          <joint_name>${joint_name}</joint_name>
+          <topic>/gz_gripper_mimic/${joint_name}</topic>
+          <p_gain>3.0</p_gain>
+          <d_gain>0.2</d_gain>
+          <i_gain>0.0</i_gain>
+          <cmd_max>50.0</cmd_max>
+          <cmd_min>-50.0</cmd_min>
+        </plugin>
+      </gazebo>
+    </xacro:macro>
+    <xacro:gz_mimic_joint_controller joint_name="${name}_outer_finger_right_joint"/>
+    <xacro:gz_mimic_joint_controller joint_name="${name}_inner_finger_right_joint"/>
+    <xacro:gz_mimic_joint_controller joint_name="${name}_fingertip_right_joint"/>
+    <xacro:gz_mimic_joint_controller joint_name="${name}_finger_right_joint"/>
+    <xacro:gz_mimic_joint_controller joint_name="${name}_outer_finger_left_joint"/>
+    <xacro:gz_mimic_joint_controller joint_name="${name}_inner_finger_left_joint"/>
+    <xacro:gz_mimic_joint_controller joint_name="${name}_fingertip_left_joint"/>
     <!-- Gazebo config -->
     <gazebo reference="${name}_inner_finger_left_link">
