Commit message: Improved mujoco description logic

File: pal_pro_gripper_description/mujoco/mj_tags.xacro (robot description, xacro)
@@ -19,5 +19,7 @@
     </xacro:macro>
     <xacro:macro name="mj_gripper_actuators" params="side reflect">
-        <position name="${side}_position" joint="${side}_inner_finger_left_joint" kp="100" ctrlrange=" 0 0.802851 " />
+        <xacro:if value="${mj_controller == 'position' or mj_controller == 'motor'}">
+            <position name="${side}_position" joint="${side}_inner_finger_left_joint" kp="100" ctrlrange=" 0 0.802851 " />
+        </xacro:if>
     </xacro:macro>
     <xacro:macro name="mj_gripper_contact" params="side">
@@ -28,7 +30,7 @@
     </xacro:macro>
     <xacro:macro name="mj_gripper_equality" params="side anchor_r anchor_l" >
-        <connect name="${side}_r" body1="${side}_fingertip_right_link" body2="${side}_outer_finger_right_link" anchor="${anchor_r}" solref="0.005" solimp="0.95 0.99"/>
-        <connect name="${side}_l" body1="${side}_fingertip_left_link" body2="${side}_outer_finger_left_link" anchor="${anchor_l}" solref="0.005" solimp="0.95 0.99"/>
-        <joint joint1="${side}_inner_finger_left_joint" joint2="${side}_inner_finger_right_joint" polycoef="0 1 0 0 0" solref="0.005" solimp="0.95 0.99"/>
+        <connect name="${side}_r" body1="${side}_fingertip_right_link" body2="${side}_outer_finger_right_link"  active="true" anchor="${anchor_r}" solref="0.005 1" solimp="0.95 0.99 0.001"/>
+        <connect name="${side}_l" body1="${side}_fingertip_left_link" body2="${side}_outer_finger_left_link" active="true"  anchor="${anchor_l}" solref="0.005 1" solimp="0.95 0.99 0.001"/>
+        <joint joint1="${side}_inner_finger_left_joint" joint2="${side}_inner_finger_right_joint" polycoef="0 1 0 0 0" solref="0.005 1" solimp="0.95 0.99 0.001"/>
     </xacro:macro>
 </robot>

Commit message: Improved mujoco description structure

File: pal_pro_gripper_description/mujoco/mj_tags.xacro (robot description, xacro)
@@ -1,24 +1,7 @@
 <?xml version="1.0"?>
 <robot xmlns:xacro="http://ros.org/wiki/xacro" name="pal_pro_gripper">
-    <xacro:macro name="mj_gripper_common">
-      <compiler strippath="false" discardvisual="false" balanceinertia="true" angle="radian" />
-        <option integrator="implicitfast" />
-        <asset>
-            <texture type="skybox" builtin="gradient" rgb1="0.3 0.5 0.7" rgb2="0 0 0" width="512"
-                height="3072" />
-            <texture type="2d" name="groundplane" builtin="checker" mark="edge" rgb1="0.2 0.3 0.4"
-                rgb2="0.1 0.2 0.3"
-                markrgb="0.8 0.8 0.8" width="300" height="300" />
-            <material name="groundplane" texture="groundplane" texuniform="true" texrepeat="5 5"
-                reflectance="0.2" />
-        </asset>
-        <worldbody>
-            <light name="spotlight" mode="targetbody" target="base_link" pos="1 0 10" />
-            <geom name="floor" size="0 0 0.05" type="plane" material="groundplane" group="0" contype="1" conaffinity="1" friction="0.001 0.0 0.0"/>
-        </worldbody>
-    </xacro:macro>
-    <xacro:macro name="mj_gripper_actuators" params="side reflect">
-        <xacro:if value="${mj_controller == 'position' or mj_controller == 'motor'}">
-            <position name="${side}_position" joint="${side}_inner_finger_left_joint" kp="100" ctrlrange=" 0 0.802851 " />
+    <xacro:macro name="mj_gripper_actuators" params="name">
+        <xacro:if value="${mj_control == 'position' or mj_control == 'motor'}">
+            <position name="${name}_position" joint="${name}_inner_finger_left_joint" kp="100" ctrlrange=" 0 0.802851 " />
         </xacro:if>
     </xacro:macro>

File: pal_pro_gripper_description/robots/pal_pro_gripper.urdf.xacro (robot description, xacro)
@@ -7,8 +7,8 @@
     <!-- false, true -->
     <xacro:arg name="use_sim_time" default="False"/>
-     <!-- Mujoco tags -->
-    <xacro:arg name="mujoco" default="false" />
-    <xacro:arg name="mj_simulate" default="false" />
+     <!-- Mujoco args -->
+    <xacro:arg name="sim_type" default="gazebo" />
     <xacro:arg name="mj_control" default="false" />
+    <xacro:arg name="mj_world_name" default="floor" />
     <!-- PROPERTIES -->
     <xacro:property name="tool_changer" value="$(arg tool_changer)" />
@@ -16,7 +16,7 @@
     <xacro:property name="name" value="gripper"/>
     <!-- Mujoco properties -->
-    <xacro:property name="mujoco" value="$(arg mujoco)" />
-    <xacro:property name="mj_simulate" value="$(arg mj_simulate)" />
-    <xacro:property name="mj_controller" value="${mj_control if mj_control != 'false' else 'no_controller'}"/>
+    <xacro:property name="sim_type" value="$(arg sim_type)" />
+    <xacro:property name="mj_control" value="${arg mj_control}"/>
+    <xacro:property name="mj_world_name" value="$(arg mj_world_name)"/>
     <!-- INCLUDES -->
     <!-- Helpers -->
@@ -29,6 +29,4 @@
     <!-- Gazebo plugins -->
     <xacro:include filename="$(find pal_pro_gripper_description)/gazebo/gazebo.urdf.xacro" />
-    <!-- MUJOCO -->
-    <xacro:include filename="$(find pal_pro_gripper_description)/mujoco/mj_tags.xacro" />
     <!-- ROBOT DEFINITION -->
     <link name="world"/>
@@ -36,16 +34,19 @@
         <origin xyz="0.0 0.0 0.08" rpy="0 0 0" />
     </xacro:pal_pro_gripper>
-    <xacro:if value="${mujoco}">
+    <xacro:if value="${sim_type == 'mujoco' or sim_type == 'mujoco-ros2-control'}">
+        <!-- MUJOCO -->
+        <xacro:include filename="$(find pal_pro_gripper_description)/mujoco/mj_tags.xacro" />
+        <xacro:include filename="$(find pal_mujoco_scenes)/scenes/${mj_world_name}.xacro" />
         <mujoco>
             <!-- Mujoco environment -->
-            <xacro:mj_gripper_common/>
+            <xacro:mj_common light_target="base_link"/>
             <!-- Contact-->
             <xacro:mj_gripper_contact side="gripper"/>
             <!-- Actuator-->
-            <xacro:if value="${mj_simulate}">
+            <xacro:if value="${sim_type == 'mujoco'}">
                 <!-- Equality-->
                 <xacro:mj_gripper_equality side="gripper" anchor_r="0.014 -0.0015 0" anchor_l="0.014 -0.001 0"/>
                 <actuator>
-                    <xacro:mj_gripper_actuators side="gripper" reflect="1"/>
+                    <xacro:mj_gripper_actuators name="gripper"/>
                 </actuator>
             </xacro:if>

Commit message: changed xacro parameter name

File: pal_pro_gripper_description/mujoco/mj_tags.xacro (robot description, xacro)
@@ -6,14 +6,14 @@
         </xacro:if>
     </xacro:macro>
-    <xacro:macro name="mj_gripper_contact" params="side">
-        <exclude body1="${side}_inner_finger_left_link"  body2="${side}_outer_finger_left_link"/>
-        <exclude body1="${side}_fingertip_left_link"     body2="${side}_outer_finger_left_link"/>
-        <exclude body1="${side}_inner_finger_right_link" body2="${side}_outer_finger_right_link"/>
-        <exclude body1="${side}_fingertip_right_link"    body2="${side}_outer_finger_right_link"/>
+    <xacro:macro name="mj_gripper_contact" params="name">
+        <exclude body1="${name}_inner_finger_left_link"  body2="${name}_outer_finger_left_link"/>
+        <exclude body1="${name}_fingertip_left_link"     body2="${name}_outer_finger_left_link"/>
+        <exclude body1="${name}_inner_finger_right_link" body2="${name}_outer_finger_right_link"/>
+        <exclude body1="${name}_fingertip_right_link"    body2="${name}_outer_finger_right_link"/>
     </xacro:macro>
-    <xacro:macro name="mj_gripper_equality" params="side anchor_r anchor_l" >
-        <connect name="${side}_r" body1="${side}_fingertip_right_link" body2="${side}_outer_finger_right_link"  active="true" anchor="${anchor_r}" solref="0.005 1" solimp="0.95 0.99 0.001"/>
-        <connect name="${side}_l" body1="${side}_fingertip_left_link" body2="${side}_outer_finger_left_link" active="true"  anchor="${anchor_l}" solref="0.005 1" solimp="0.95 0.99 0.001"/>
-        <joint joint1="${side}_inner_finger_left_joint" joint2="${side}_inner_finger_right_joint" polycoef="0 1 0 0 0" solref="0.005 1" solimp="0.95 0.99 0.001"/>
+    <xacro:macro name="mj_gripper_equality" params="name anchor_r anchor_l" >
+        <connect name="${name}_r" body1="${name}_fingertip_right_link" body2="${name}_outer_finger_right_link"  active="true" anchor="${anchor_r}" solref="0.005 1" solimp="0.95 0.99 0.001"/>
+        <connect name="${name}_l" body1="${name}_fingertip_left_link" body2="${name}_outer_finger_left_link" active="true"  anchor="${anchor_l}" solref="0.005 1" solimp="0.95 0.99 0.001"/>
+        <joint joint1="${name}_inner_finger_left_joint" joint2="${name}_inner_finger_right_joint" polycoef="0 1 0 0 0" solref="0.005 1" solimp="0.95 0.99 0.001"/>
     </xacro:macro>
 </robot>
