Commit message: add working mimic joint configuration

File: pal_pro_gripper_description/ros2_control/ros2_control.urdf.xacro (robot description, xacro)
@@ -26,5 +26,5 @@
       </hardware>
       <!-- pal-pro-gripper -->
-      <xacro:ros2_control_pal_pro_gripper name="gripper_finger" reduction="1.0" />
+      <xacro:ros2_control_pal_pro_gripper name="gripper" reduction="1.0" />
     </ros2_control>
   </xacro:macro>

File: pal_pro_gripper_description/urdf/pal_pro_gripper.ros2_control.xacro (robot description, xacro)
@@ -14,5 +14,5 @@
 <robot xmlns:xacro="http://ros.org/wiki/xacro">
   <xacro:macro name="ros2_control_pal_pro_gripper" params="name reduction" >
-    <joint name="${name}_joint">
+    <joint name="${name}_finger_joint">
       <command_interface name="position"/>
       <state_interface name="position">
@@ -22,6 +22,6 @@
       <state_interface name="effort"/>
     </joint>
-    <joint name="${name}_outer_finger_left_joint">
-      <param name="mimic">${name}_joint</param>
+    <joint name="${name}_outer_finger_right_joint">
+      <param name="mimic">${name}_finger_joint</param>
       <param name="multiplier">1</param>
       <command_interface name="position" />
@@ -30,7 +30,31 @@
       <state_interface name="effort" />
     </joint>
-    <joint name="${name}_outer_finger_right_joint">
-      <param name="mimic">${name}_joint</param>
+    <joint name="${name}_inner_finger_left_joint">
+      <param name="mimic">${name}_finger_joint</param>
       <param name="multiplier">1</param>
+      <command_interface name="position" />
+      <state_interface name="position" />
+      <state_interface name="velocity" />
+      <state_interface name="effort" />
+    </joint>
+    <joint name="${name}_inner_finger_right_joint">
+      <param name="mimic">${name}_finger_joint</param>
+      <param name="multiplier">1</param>
+      <command_interface name="position" />
+      <state_interface name="position" />
+      <state_interface name="velocity" />
+      <state_interface name="effort" />
+    </joint>
+    <joint name="${name}_fingertip_right_joint">
+      <param name="mimic">${name}_finger_joint</param>
+      <param name="multiplier">-1</param>
+      <command_interface name="position" />
+      <state_interface name="position" />
+      <state_interface name="velocity" />
+      <state_interface name="effort" />
+    </joint>
+    <joint name="${name}_fingertip_left_joint">
+      <param name="mimic">${name}_finger_joint</param>
+      <param name="multiplier">-1</param>
       <command_interface name="position" />
       <state_interface name="position" />
@@ -41,5 +65,5 @@
     joint-->
     <xacro:include filename="$(find pal_pro_gripper_description)/urdf/pro_gripper.transmission.xacro" />
-    <xacro:pal_pro_gripper_transmission name="${name}"/>
+    <xacro:pal_pro_gripper_transmission name="${name}_finger"/>
   </xacro:macro>
 </robot>

File: pal_pro_gripper_description/urdf/pro_gripper.urdf.xacro (robot description, xacro)
@@ -1,7 +1,4 @@
 <?xml version="1.0"?>
 <robot xmlns:xacro="http://ros.org/wiki/xacro">
-  <!--File
-  includes-->
-  <!-- TODO: grasping frames -->
   <xacro:macro name="pro_finger" params="name side reflect">
     <link name="${name}_inner_finger_${side}_link">
@@ -37,9 +34,4 @@
       <mimic joint="${name}_finger_joint" multiplier="1" offset="0" />
     </joint>
-    <!-- Mimic finger joint
-     <xacro:mimic_joint_plugin_gazebo name="${name}_${side}_mimic_pro_gripper_1"
-      parent_joint="${name}_finger_joint" mimic_joint="${name}_inner_finger_${side}_joint"
-      has_pid="false" multiplier="1.0" offset="0" />
-    -->
     <link name="${name}_outer_finger_${side}_link">
       <inertial>
@@ -83,11 +75,4 @@
       </xacro:unless>
     </joint>
-    <!--  The left outer joint is set as gripper_finger_joint. All other joints are passive and will
-    mimic this joint-->
-    <xacro:unless value="${side == 'left'}">
-      <!--<xacro:mimic_joint_plugin_gazebo name="${name}_${side}_mimic_pro_gripper_2"
-        parent_joint="${name}_finger_joint" mimic_joint="${name}_outer_finger_${side}_joint"
-        has_pid="false" multiplier="1.0" offset="0.0" />-->
-    </xacro:unless>
     <link name="${name}_fingertip_${side}_link">
       <inertial>
@@ -121,8 +106,4 @@
       <mimic joint="${name}_finger_joint" multiplier="-1" offset="0" />
     </joint>
-    <!-- Mimic finger joint
-    <xacro:mimic_joint_plugin_gazebo name="${name}_${side}_mimic_pro_gripper_3"
-      parent_joint="${name}_finger_joint" mimic_joint="${name}_fingertip_${side}_joint"
-      has_pid="false" multiplier="-1.0" offset="0.0" />-->
   </xacro:macro>
   <xacro:macro name="pal_pro_gripper" params="name parent *origin">

Commit message: Add missing sim_type xacro args

File: pal_pro_gripper_description/ros2_control/ros2_control.urdf.xacro (robot description, xacro)
@@ -13,5 +13,5 @@
  -->
 <robot xmlns:xacro="http://ros.org/wiki/xacro" name="pal_pro_gripper">
-  <xacro:macro name="pal_pro_gripper_ros2_control">
+  <xacro:macro name="pal_pro_gripper_ros2_control" params="use_sim_time:=^|false sim_type:=no-simulation">
     <xacro:include filename="$(find pal_pro_gripper_description)/urdf/gripper.ros2_control.xacro" />
     <ros2_control name="ros2_control_pal_pro_gripper_system" type="system">

File: pal_pro_gripper_description/urdf/gripper.ros2_control.xacro (robot description, xacro)
@@ -13,6 +13,6 @@
 -->
 <robot xmlns:xacro="http://ros.org/wiki/xacro">
-  <xacro:macro name="ros2_control_pal_pro_gripper" params="name reduction">
-    <xacro:macro name="ros2_control_pal_pro_gripper_mimic_joint" params="mimic_joint_name actuated_joint_name multiplier">
+  <xacro:macro name="ros2_control_pal_pro_gripper" params="name reduction sim_type:=no-simulation">
+    <xacro:macro name="ros2_control_pal_pro_gripper_mimic_joint" params="mimic_joint_name actuated_joint_name multiplier sim_type:=no-simulation">
       <joint name="${mimic_joint_name}">
         <param name="mimic">${actuated_joint_name}</param>
