Commit message: Update mimicjoint and typos

File: pal_pro_gripper_description/robots/pal_pro_gripper.urdf.xacro (robot description, xacro)
@@ -2,10 +2,10 @@
 <robot name="pal_pro_gripper" xmlns:xacro="http://ros.org/wiki/xacro">
     <xacro:include filename="$(find pal_pro_gripper_description)/urdf/pro_gripper.urdf.xacro" />
-    <xacro:property name="prefix" value="gripper"/>
-    <gazebo>
+    <xacro:property name="name" value="gripper"/>
+    <!-- <gazebo>
         <plugin name="gazebo_ros_control" filename="libgazebo_ros_control.so">
             <robotNamespace></robotNamespace>
         </plugin>
-    </gazebo>
+    </gazebo> -->
     <link name="world"/>
     <joint name="world_fixed" type="fixed">
@@ -35,6 +35,6 @@
         </inertial>
     </link>
-    <xacro:pal_pro_gripper name="${prefix}" parent="gripper_root_link" >
-        <origin xyz="0.05 0 0.85" rpy="0 1.5708 0"/>
+    <xacro:pal_pro_gripper name="${name}" parent="gripper_root_link" >
+        <origin xyz="0.1 0 0.85" rpy="0 1.5708 0"/>
     </xacro:pal_pro_gripper>
 </robot>

File: pal_pro_gripper_description/urdf/materials.urdf.xacro (robot description, xacro)
@@ -8,9 +8,9 @@
 -->
 <robot>
-  <material name="Grey">
+  <!-- <material name="Grey">
     <color rgba="0.75294 0.75294 0.75294 1"/>
   </material>
   <material name="White">
     <color rgba="1 1 1 1"/>
-  </material>
+  </material> -->
 </robot>

File: pal_pro_gripper_description/urdf/pro_gripper.urdf.xacro (robot description, xacro)
@@ -39,10 +39,11 @@
       <child link="${name}_inner_finger_${side}_link" />
       <axis xyz="0 0 -1" />
-      <limit lower="-0.2618" upper="0" effort="0" velocity="0" />
+      <limit lower="0" upper="0.81" velocity="2" effort="0.1" />
+      <mimic joint="${name}_finger_joint" multiplier="1" offset="0" />
     </joint>
     <!-- Mimic finger joint-->
     <xacro:mimic_joint_plugin_gazebo name="${name}_${side}_mimic_pro_gripper_1"
       parent_joint="${name}_finger_joint" mimic_joint="${name}_inner_finger_${side}_joint"
-      has_pid="false" multiplier="1.0" offset="0.0" />
+      has_pid="false" multiplier="1.0" offset="0.15" />
     <link name="${name}_outer_finger_${side}_link">
       <inertial>
@@ -78,5 +79,11 @@
       <child link="${name}_outer_finger_${side}_link" />
       <axis xyz="0 0 -1" />
-      <limit lower="0" upper="0" effort="0" velocity="0" />
+      <limit lower="0" upper="0.6" velocity="2" effort="0.1" />
+      <xacro:if value="${side == 'left'}">
+            <dynamics damping="0.03"/>
+      </xacro:if>
+      <xacro:unless value="${side == 'left'}">
+            <mimic joint="${name}_finger_joint" multiplier="1" offset="0" />
+      </xacro:unless>
     </joint>
     <!--  The left outer joint is set as gripper_finger_joint. All other joints are passive and will
@@ -115,5 +122,6 @@
       <child link="${name}_fingertip_${side}_link" />
       <axis xyz="0 0 -1" />
-      <limit lower="0" upper="0" effort="0" velocity="0" />
+      <limit lower="-0.8757" upper="0" velocity="2" effort="0.1" />
+      <mimic joint="${name}_finger_joint" multiplier="-1" offset="0" />
     </joint>
     <!-- Mimic finger joint-->
@@ -152,10 +160,14 @@
       <axis xyz="0 0 0" />
     </joint>
-    <xacro:pro_finger name="${name}" side='left' reflect="1" />
-    <xacro:pro_finger name="${name}" side='right' reflect="-1" />
+    <gazebo reference="${name}_finger_joint">
+      <implicitSpringDamper>1</implicitSpringDamper>
+      <provideFeedback>1</provideFeedback>
+    </gazebo>
+    <xacro:pro_finger name="${name}" side="left" reflect="1" />
+    <xacro:pro_finger name="${name}" side="right" reflect="-1" />
     <!-- Transmission only set to left outer finger joint, other joints are passive and mimic this
     joint-->
     <xacro:pal_pro_gripper_transmission name="${name}" />
-    <xacro:gazebo_gripper_grasp name="${name}_grasp" palm_link="${parent}" finger_link_left="${name}_inner_finger_left_link" finger_link_right="${name}_inner_finger_right_link" />
+    <xacro:gazebo_gripper_grasp name="${name}_grasp" palm_link="${parent}" finger_link_left="${name}_outer_finger_left_link" finger_link_right="${name}_outer_finger_right_link" />
   </xacro:macro>
 </robot>

Commit message: remove materials to make use of pal_urdf_utils package

File: pal_pro_gripper_description/robots/pal_pro_gripper.urdf.xacro (robot description, xacro)
@@ -1,8 +1,9 @@
 <?xml version="1.0" ?>
 <robot name="pal_pro_gripper" xmlns:xacro="http://ros.org/wiki/xacro">
+    <!--File includes-->
+    <xacro:include filename="$(find pal_urdf_utils)/urdf/deg_to_rad.xacro" />
+    <xacro:include filename="$(find pal_urdf_utils)/urdf/materials.urdf.xacro" />
     <xacro:include filename="$(find pal_pro_gripper_description)/urdf/pro_gripper.urdf.xacro" />
     <xacro:property name="name" value="gripper"/>
-    <!-- Materials for visualization -->
-    <xacro:include filename="$(find pal_pro_gripper_description)/urdf/materials.urdf.xacro" />
     <!-- Load gazebo plugins -->
     <xacro:include filename="$(find pal_pro_gripper_description)/gazebo/gazebo.urdf.xacro" />
@@ -34,4 +35,9 @@
         </inertial>
     </link>
+    <gazebo reference="gripper_root_link">
+      <material>Gazebo/DarkGrey</material>
+      <mu1>0.9</mu1>
+      <mu2>0.9</mu2>
+    </gazebo>
     <xacro:pal_pro_gripper name="${name}" parent="gripper_root_link" >
         <origin xyz="0.1 0 0.85" rpy="0 1.5708 0"/>

File: pal_pro_gripper_description/urdf/pro_gripper.urdf.xacro (robot description, xacro)
@@ -3,5 +3,4 @@
   <!--File
   includes-->
-  <xacro:include filename="$(find pal_pro_gripper_description)/urdf/deg_to_rad.urdf.xacro" />
   <xacro:include filename="$(find pal_pro_gripper_description)/urdf/pro_gripper.transmission.xacro" />
   <!-- Gazebo simulation plugins -->
@@ -23,5 +22,5 @@
           <mesh filename="package://pal_pro_gripper_description/meshes/inner_finger.stl" />
         </geometry>
-        <material name="Grey" />
+        <material name="White" />
       </visual>
       <collision>
@@ -107,5 +106,5 @@
           <mesh filename="package://pal_pro_gripper_description/meshes/fingertip.stl" />
         </geometry>
-        <material name="Grey" />
+        <material name="White" />
       </visual>
       <collision>
@@ -144,5 +143,5 @@
           <mesh filename="package://pal_pro_gripper_description/meshes/base_link.stl" />
         </geometry>
-        <material name="Grey" />
+        <material name="pal/DarkGrey" />
       </visual>
       <collision>
@@ -159,4 +158,39 @@
       <axis xyz="0 0 0" />
     </joint>
+    <gazebo reference="${name}_inner_finger_left_link">
+      <material>Gazebo/White</material>
+      <mu1>0.9</mu1>
+      <mu2>0.9</mu2>
+    </gazebo>
+    <gazebo reference="${name}_inner_finger_right_link">
+      <material>Gazebo/White</material>
+      <mu1>0.9</mu1>
+      <mu2>0.9</mu2>
+    </gazebo>
+    <gazebo reference="${name}_outer_finger_left_link">
+      <material>Gazebo/White</material>
+      <mu1>0.9</mu1>
+      <mu2>0.9</mu2>
+    </gazebo>
+    <gazebo reference="${name}_outer_finger_right_link">
+      <material>Gazebo/White</material>
+      <mu1>0.9</mu1>
+      <mu2>0.9</mu2>
+    </gazebo>
+    <gazebo reference="${name}_fingertip_right_link">
+      <material>Gazebo/White</material>
+      <mu1>0.9</mu1>
+      <mu2>0.9</mu2>
+    </gazebo>
+    <gazebo reference="${name}_fingertip_left_link">
+      <material>Gazebo/White</material>
+      <mu1>0.9</mu1>
+      <mu2>0.9</mu2>
+    </gazebo>
+    <gazebo reference="${name}_base_link">
+      <material>Gazebo/DarkGrey</material>
+      <mu1>0.9</mu1>
+      <mu2>0.9</mu2>
+    </gazebo>
     <gazebo reference="${name}_finger_joint">
       <implicitSpringDamper>1</implicitSpringDamper>

Commit message: box support for the gripper reduced

File: pal_pro_gripper_description/robots/pal_pro_gripper.urdf.xacro (robot description, xacro)
@@ -12,38 +12,14 @@
     <xacro:include filename="$(find pal_pro_gripper_description)/ros2_control/ros2_control.urdf.xacro" />
     <xacro:pal_pro_gripper_ros2_control use_sim="$(arg use_sim)" />
-    <link name="world"/>
-    <joint name="world_fixed" type="fixed">
-        <origin xyz="0 0 0" rpy="0 0 0"/>
-        <parent link="world"/>
-        <child link="gripper_root_link"/>
-    </joint>
     <link name="gripper_root_link">
         <visual>
-            <origin xyz="0 0 0.5" rpy="0 0 0"/>
+            <origin xyz="0 0 0" rpy="0 0 0"/>
             <geometry>
-                <box size="0.1 0.1 1.0"/>
+                <box size="0.01 0.01 0.01"/>
             </geometry>
         </visual>
-        <collision>
-            <origin xyz="0 0 0.5" rpy="0 0 0"/>
-            <geometry>
-                <box size="0.1 0.1 1.0"/>
-            </geometry>
-        </collision>
-        <inertial>
-            <mass value="1e2" />
-            <origin xyz="0.0 0.0 0.0" />
-            <inertia ixx = "0.000001" ixy = "0.000000" ixz = "0.000000"
-                     iyx = "0.000000" iyy = "0.000001" iyz = "0.000000"
-                     izx = "0.000000" izy = "0.000000" izz = "0.000001" />
-        </inertial>
     </link>
-    <gazebo reference="gripper_root_link">
-      <material>Gazebo/DarkGrey</material>
-      <mu1>0.9</mu1>
-      <mu2>0.9</mu2>
-    </gazebo>
     <xacro:pal_pro_gripper name="${name}" parent="gripper_root_link" >
-        <origin xyz="0.1 0 0.85" rpy="0 1.5708 0"/>
+        <origin xyz="0.0 0.0 0.07" rpy="0 0 0"/>
     </xacro:pal_pro_gripper>
 </robot>

Commit message: add world_link to improve the spawn in simulation

File: pal_pro_gripper_description/robots/pal_pro_gripper.urdf.xacro (robot description, xacro)
@@ -12,14 +12,33 @@
     <xacro:include filename="$(find pal_pro_gripper_description)/ros2_control/ros2_control.urdf.xacro" />
     <xacro:pal_pro_gripper_ros2_control use_sim="$(arg use_sim)" />
+    <link name="world"/>
+    <joint name="world_fixed" type="fixed">
+        <origin xyz="0 0 0" rpy="0 0 0"/>
+        <parent link="world"/>
+        <child link="gripper_root_link"/>
+    </joint>
     <link name="gripper_root_link">
         <visual>
-            <origin xyz="0 0 0" rpy="0 0 0"/>
+            <origin xyz="0 0 0.02" rpy="0 0 0"/>
             <geometry>
                 <box size="0.01 0.01 0.01"/>
             </geometry>
         </visual>
+        <collision>
+            <origin xyz="0 0 0.2" rpy="0 0 0"/>
+            <geometry>
+                <box size="0.01 0.01 0.05"/>
+            </geometry>
+        </collision>
+        <inertial>
+            <mass value="1e2" />
+            <origin xyz="0.0 0.0 0.0" />
+            <inertia ixx = "0.000001" ixy = "0.000000" ixz = "0.000000"
+                     iyx = "0.000000" iyy = "0.000001" iyz = "0.000000"
+                     izx = "0.000000" izy = "0.000000" izz = "0.000001" />
+        </inertial>
     </link>
-    <xacro:pal_pro_gripper name="${name}" parent="gripper_root_link" >
-        <origin xyz="0.0 0.0 0.07" rpy="0 0 0"/>
+    <xacro:pal_pro_gripper name="${name}" parent="gripper_root_link">
+        <origin xyz="0.0 0.0 0.08" rpy="0 0 0"/>
     </xacro:pal_pro_gripper>
 </robot>

Commit message: fix collision of the little box support

File: pal_pro_gripper_description/robots/pal_pro_gripper.urdf.xacro (robot description, xacro)
@@ -26,7 +26,7 @@
         </visual>
         <collision>
-            <origin xyz="0 0 0.2" rpy="0 0 0"/>
+            <origin xyz="0 0 0.02" rpy="0 0 0"/>
             <geometry>
-                <box size="0.01 0.01 0.05"/>
+                <box size="0.01 0.01 0.01"/>
             </geometry>
         </collision>

Commit message: simplify the root link adding a world link

File: pal_pro_gripper_description/robots/pal_pro_gripper.urdf.xacro (robot description, xacro)
@@ -13,32 +13,6 @@
     <xacro:pal_pro_gripper_ros2_control use_sim="$(arg use_sim)" />
     <link name="world"/>
-    <joint name="world_fixed" type="fixed">
-        <origin xyz="0 0 0" rpy="0 0 0"/>
-        <parent link="world"/>
-        <child link="gripper_root_link"/>
-    </joint>
-    <link name="gripper_root_link">
-        <visual>
-            <origin xyz="0 0 0.02" rpy="0 0 0"/>
-            <geometry>
-                <box size="0.01 0.01 0.01"/>
-            </geometry>
-        </visual>
-        <collision>
-            <origin xyz="0 0 0.02" rpy="0 0 0"/>
-            <geometry>
-                <box size="0.01 0.01 0.01"/>
-            </geometry>
-        </collision>
-        <inertial>
-            <mass value="1e2" />
-            <origin xyz="0.0 0.0 0.0" />
-            <inertia ixx = "0.000001" ixy = "0.000000" ixz = "0.000000"
-                     iyx = "0.000000" iyy = "0.000001" iyz = "0.000000"
-                     izx = "0.000000" izy = "0.000000" izz = "0.000001" />
-        </inertial>
-    </link>
-    <xacro:pal_pro_gripper name="${name}" parent="gripper_root_link">
-        <origin xyz="0.0 0.0 0.08" rpy="0 0 0"/>
+    <xacro:pal_pro_gripper name="${name}" parent="world">
+        <origin xyz="0.0 0.0 0.08" rpy="0 0 0" />
     </xacro:pal_pro_gripper>
 </robot>

Commit message: Gripper std with tool_changer new arg

File: pal_pro_gripper_description/robots/pal_pro_gripper.urdf.xacro (robot description, xacro)
@@ -1,18 +1,30 @@
 <?xml version="1.0" ?>
-<robot name="pal_pro_gripper" xmlns:xacro="http://ros.org/wiki/xacro">
-    <!--File includes-->
+<robot name="pal_pro_gripper"
+    xmlns:xacro="http://ros.org/wiki/xacro">
+    <!-- ARGUMENTS  -->
+    <!-- False, True -->
+    <xacro:arg name="tool_changer" default="False"/>
+    <!-- false, true -->
+    <xacro:arg name="use_sim_time" default="False"/>
+    <!-- PROPERTIES -->
+    <xacro:property name="tool_changer" value="$(arg tool_changer)" />
+    <xacro:property name="use_sim_time" value="$(arg use_sim_time)" />
+    <xacro:property name="name" value="gripper"/>
+    <!-- INCLUDES -->
+    <!-- Helpers -->
     <xacro:include filename="$(find pal_urdf_utils)/urdf/deg_to_rad.urdf.xacro" />
     <xacro:include filename="$(find pal_urdf_utils)/urdf/materials.urdf.xacro" />
-    <xacro:include filename="$(find pal_pro_gripper_description)/urdf/pro_gripper.urdf.xacro" />
-    <!-- Load gazebo plugins -->
+    <!-- Gripper -->
+    <xacro:include filename="$(find pal_pro_gripper_description)/urdf/gripper.urdf.xacro" />
+    <!-- ROS 2 control-->
+    <xacro:include filename="$(find pal_pro_gripper_description)/ros2_control/ros2_control.urdf.xacro" />
+    <!-- Gazebo plugins -->
     <xacro:include filename="$(find pal_pro_gripper_description)/gazebo/gazebo.urdf.xacro" />
-    <xacro:property name="name" value="gripper"/>
-    <xacro:arg name="use_sim" default="false"/>
-    <!-- ros2_control -->
-    <xacro:include filename="$(find pal_pro_gripper_description)/ros2_control/ros2_control.urdf.xacro" />
-    <xacro:pal_pro_gripper_ros2_control use_sim="$(arg use_sim)" />
+    <!-- ROBOT DEFINITION -->
     <link name="world"/>
-    <xacro:pal_pro_gripper name="${name}" parent="world">
+    <xacro:pal_pro_gripper tool_changer="${tool_changer}" name="${name}" parent="world">
         <origin xyz="0.0 0.0 0.08" rpy="0 0 0" />
     </xacro:pal_pro_gripper>
+    <!-- ROS 2 Control -->
+    <xacro:pal_pro_gripper_ros2_control />
 </robot>

File: pal_pro_gripper_description/ros2_control/ros2_control.urdf.xacro (robot description, xacro)
@@ -12,14 +12,13 @@
   limitations under the License.
  -->
-<robot xmlns:xacro="http://ros.org/wiki/xacro"
-       name="pal_pro_gripper" >
-    <xacro:macro name="pal_pro_gripper_ros2_control" params="use_sim:=^|false">
-    <xacro:include filename="$(find pal_pro_gripper_description)/urdf/pal_pro_gripper.ros2_control.xacro" />
+<robot xmlns:xacro="http://ros.org/wiki/xacro" name="pal_pro_gripper">
+  <xacro:macro name="pal_pro_gripper_ros2_control">
+    <xacro:include filename="$(find pal_pro_gripper_description)/urdf/gripper.ros2_control.xacro" />
     <ros2_control name="ros2_control_pal_pro_gripper_system" type="system">
       <hardware>
-        <xacro:if value="$(arg use_sim)">
+        <xacro:if value="${use_sim_time}">
           <plugin>gazebo_ros2_control/GazeboSystem</plugin>
         </xacro:if>
-        <xacro:unless value="$(arg use_sim)">
+        <xacro:unless value="${use_sim_time}">
           <plugin>robot_control/RobotControl</plugin>
         </xacro:unless>

Commit message: Added mujoco model description

File: pal_pro_gripper_description/robots/pal_pro_gripper.urdf.xacro (robot description, xacro)
@@ -7,8 +7,16 @@
     <!-- false, true -->
     <xacro:arg name="use_sim_time" default="False"/>
+     <!-- Mujoco tags -->
+    <xacro:arg name="mujoco" default="false" />
+    <xacro:arg name="mj_simulate" default="false" />
+    <xacro:arg name="mj_control" default="false" />
     <!-- PROPERTIES -->
     <xacro:property name="tool_changer" value="$(arg tool_changer)" />
     <xacro:property name="use_sim_time" value="$(arg use_sim_time)" />
     <xacro:property name="name" value="gripper"/>
+    <!-- Mujoco properties -->
+    <xacro:property name="mujoco" value="$(arg mujoco)" />
+    <xacro:property name="mj_simulate" value="$(arg mj_simulate)" />
+    <xacro:property name="mj_controller" value="${mj_control if mj_control != 'false' else 'no_controller'}"/>
     <!-- INCLUDES -->
     <!-- Helpers -->
@@ -21,4 +29,6 @@
     <!-- Gazebo plugins -->
     <xacro:include filename="$(find pal_pro_gripper_description)/gazebo/gazebo.urdf.xacro" />
+    <!-- MUJOCO -->
+    <xacro:include filename="$(find pal_pro_gripper_description)/mujoco/mj_tags.xacro" />
     <!-- ROBOT DEFINITION -->
     <link name="world"/>
@@ -26,4 +36,20 @@
         <origin xyz="0.0 0.0 0.08" rpy="0 0 0" />
     </xacro:pal_pro_gripper>
+    <xacro:if value="${mujoco}">
+        <mujoco>
+            <!-- Mujoco environment -->
+            <xacro:mj_gripper_common/>
+            <!-- Contact-->
+            <xacro:mj_gripper_contact side="gripper"/>
+            <!-- Actuator-->
+            <xacro:if value="${mj_simulate}">
+                <!-- Equality-->
+                <xacro:mj_gripper_equality side="gripper" anchor_r="0.014 -0.0015 0" anchor_l="0.014 -0.001 0"/>
+                <actuator>
+                    <xacro:mj_gripper_actuators side="gripper" reflect="1"/>
+                </actuator>
+            </xacro:if>
+        </mujoco>
+    </xacro:if>
     <!-- ROS 2 Control -->
     <xacro:pal_pro_gripper_ros2_control />

Commit message: changed world and mujoco xacro argument name

File: pal_pro_gripper_description/robots/pal_pro_gripper.urdf.xacro (robot description, xacro)
@@ -10,5 +10,5 @@
     <xacro:arg name="sim_type" default="gazebo" />
     <xacro:arg name="mj_control" default="false" />
-    <xacro:arg name="mj_world_name" default="floor" />
+    <xacro:arg name="world_name" default="floor" />
     <!-- PROPERTIES -->
     <xacro:property name="tool_changer" value="$(arg tool_changer)" />
@@ -18,5 +18,5 @@
     <xacro:property name="sim_type" value="$(arg sim_type)" />
     <xacro:property name="mj_control" value="${arg mj_control}"/>
-    <xacro:property name="mj_world_name" value="$(arg mj_world_name)"/>
+    <xacro:property name="world_name" value="$(arg world_name)"/>
     <!-- INCLUDES -->
     <!-- Helpers -->
@@ -37,14 +37,14 @@
         <!-- MUJOCO -->
         <xacro:include filename="$(find pal_pro_gripper_description)/mujoco/mj_tags.xacro" />
-        <xacro:include filename="$(find pal_mujoco_scenes)/scenes/${mj_world_name}.xacro" />
+        <xacro:include filename="$(find pal_mujoco_scenes)/scenes/${world_name}.xacro" />
         <mujoco>
             <!-- Mujoco environment -->
             <xacro:mj_common light_target="base_link"/>
             <!-- Contact-->
-            <xacro:mj_gripper_contact side="gripper"/>
+            <xacro:mj_gripper_contact name="gripper"/>
             <!-- Actuator-->
             <xacro:if value="${sim_type == 'mujoco'}">
                 <!-- Equality-->
-                <xacro:mj_gripper_equality side="gripper" anchor_r="0.014 -0.0015 0" anchor_l="0.014 -0.001 0"/>
+                <xacro:mj_gripper_equality name="gripper" anchor_r="0.014 -0.0015 0" anchor_l="0.014 -0.001 0"/>
                 <actuator>
                     <xacro:mj_gripper_actuators name="gripper"/>

Commit message: fixing sim_type

File: pal_pro_gripper_description/robots/pal_pro_gripper.urdf.xacro (robot description, xacro)
@@ -17,5 +17,5 @@
     <!-- Mujoco properties -->
     <xacro:property name="sim_type" value="$(arg sim_type)" />
-    <xacro:property name="mj_control" value="${arg mj_control}"/>
+    <xacro:property name="mj_control" value="$(arg mj_control)"/>
     <xacro:property name="world_name" value="$(arg world_name)"/>
     <!-- INCLUDES -->

File: pal_pro_gripper_description/urdf/gripper.ros2_control.xacro (robot description, xacro)
@@ -31,5 +31,5 @@
     <xacro:ros2_control_pal_pro_gripper_mimic_joint mimic_joint_name="${name}_inner_finger_right_joint" actuated_joint_name="${name}_finger_joint" multiplier="1"/>
     <xacro:ros2_control_pal_pro_gripper_mimic_joint mimic_joint_name="${name}_fingertip_right_joint" actuated_joint_name="${name}_finger_joint" multiplier="-1"/>
-    <xacro:ros2_control_pal_pro_gripper_mimic_joint mimic_joint_name="${name}_inner_finger_left_joint" actuated_joint_name="${name}_finger_joint" multiplier="1}"/>
+    <xacro:ros2_control_pal_pro_gripper_mimic_joint mimic_joint_name="${name}_inner_finger_left_joint" actuated_joint_name="${name}_finger_joint" multiplier="1"/>
     <xacro:ros2_control_pal_pro_gripper_mimic_joint mimic_joint_name="${name}_fingertip_left_joint" actuated_joint_name="${name}_finger_joint" multiplier="-1"/>
     <!-- Transmission only set to left finger joint, other joints are passive and mimic this

File: pal_pro_gripper_description/urdf/gripper.urdf.xacro (robot description, xacro)
@@ -32,5 +32,5 @@
     <!-- Outer finger -->
     <link name="${name}_outer_finger_${side}_link">
-      <xacro:inertial_outer_finger_link/>
+      <xacro:inertial_outer_finger_link />
       <visual>
         <origin xyz="0 0 0" rpy="0 0 0" />
