Commit message: adding calibration_tool

File: pal_pro_gripper_description/robots/pal_pro_gripper.urdf.xacro (robot description, xacro)
@@ -13,4 +13,5 @@
     <!-- PROPERTIES -->
     <xacro:property name="tool_changer" value="$(arg tool_changer)" />
+    <xacro:property name="calibration_tool" value="z$(arg calibration_tool)" />
     <xacro:property name="use_sim_time" value="$(arg use_sim_time)" />
     <xacro:property name="name" value="gripper"/>
@@ -31,5 +32,5 @@
     <!-- ROBOT DEFINITION -->
     <link name="world"/>
-    <xacro:pal_pro_gripper tool_changer="${tool_changer}" name="${name}" parent="world">
+    <xacro:pal_pro_gripper tool_changer="${tool_changer}" name="${name}" parent="world" calibration_tool="${calibration_tool}">
         <origin xyz="0.0 0.0 0.08" rpy="0 0 0" />
     </xacro:pal_pro_gripper>

File: pal_pro_gripper_description/urdf/gripper.urdf.xacro (robot description, xacro)
@@ -128,5 +128,5 @@
   </xacro:macro>
   <!-- GRIPPER DEFINITION -->
-  <xacro:macro name="pal_pro_gripper" params="tool_changer:=False name parent *origin">
+  <xacro:macro name="pal_pro_gripper" params="tool_changer:=False name parent *origin calibration_tool:=False">
     <!-- Vesion name depending if it is a prototype -->
     <xacro:property name="gripper_base_type" value="${'base_link_tc' if tool_changer else 'base_link_ntc'}" />
@@ -163,15 +163,50 @@
     </joint>
     <!-- Grasping Frame -->
-    <joint name="${name}_grasping_frame_joint" type="fixed">
-      <parent link="${name}_base_link"/>
-      <child link="${name}_grasping_link"/>
-      <origin xyz="0.0 0 0.157157" rpy="0 -1.57 0" />
-    </joint>
-    <link name="${name}_grasping_link">
-      <inertial>
-        <mass value="1e-9" />
-        <inertia ixx="1e-9" ixy="0.0" ixz="0.0" iyy="1e-9" iyz="0.0" izz="1e-9" />
-      </inertial>
-    </link>
+    <xacro:if value="${calibration_tool}">
+      <joint name="${name}_grasping_frame_joint" type="fixed">
+        <parent link="${name}_base_link"/>
+        <child link="${name}_grasping_link"/>
+        <origin xyz="0.0 0.0 0.13" rpy="0 0 0" />
+      </joint>
+      <link name="${name}_grasping_link">
+        <inertial>
+          <mass value="0.1" />
+          <origin xyz="0 0 0.1" rpy="0 0 0" />
+          <inertia ixx="0.000341" ixy="0" ixz="0" iyy="0.000241" iyz="0" izz="0.000101" />
+        </inertial>
+        <visual>
+          <origin xyz="0 0 0.1" rpy="0 0 0" />
+          <geometry>
+            <box size="0.01 0.12 0.09" />
+          </geometry>
+          <material name="grasp_box_color">
+            <color rgba="0 0 1 1" />
+          </material>
+        </visual>
+        <collision>
+          <origin xyz="0 0 0.1" rpy="0 0 0" />
+          <geometry>
+            <box size="0.01 0.12 0.09" />
+          </geometry>
+        </collision>
+      </link>
+      <gazebo reference="${name}_grasping_link">
+        <material>Gazebo/Blue</material>
+        <turnGravityOff>true</turnGravityOff>
+      </gazebo>
+    </xacro:if>
+    <xacro:unless value="${calibration_tool}">
+      <joint name="${name}_grasping_frame_joint" type="fixed">
+        <parent link="${name}_base_link"/>
+        <child link="${name}_grasping_link"/>
+        <origin xyz="0.0 0.0 0.157157" rpy="0 -1.57 0" />
+      </joint>
+      <link name="${name}_grasping_link">
+        <inertial>
+          <mass value="1e-9" />
+          <inertia ixx="1e-9" ixy="0.0" ixz="0.0" iyy="1e-9" iyz="0.0" izz="1e-9" />
+        </inertial>
+      </link>
+    </xacro:unless>
     <!-- Fingers -->
     <xacro:pro_finger name="${name}" side="left" reflect="-1" finger_offset="${finger_offset}"/>

Commit message: Fix a typo

File: pal_pro_gripper_description/robots/pal_pro_gripper.urdf.xacro (robot description, xacro)
@@ -13,5 +13,5 @@
     <!-- PROPERTIES -->
     <xacro:property name="tool_changer" value="$(arg tool_changer)" />
-    <xacro:property name="calibration_tool" value="z$(arg calibration_tool)" />
+    <xacro:property name="calibration_tool" value="$(arg calibration_tool)" />
     <xacro:property name="use_sim_time" value="$(arg use_sim_time)" />
     <xacro:property name="name" value="gripper"/>
