Commit message: Fix gripper mimic joints getting stuck on their limit in Gazebo
gz_ros2_control's mimic controller can overshoot a joint into its limit and never recover (unfixed DART bug on Harmonic, see ros-controls/gz_ros2_control#165). Mimic joints are now independently actuated in simulation instead (real robot unaffected), with gripper_grasper_srv computing their target positions from the URDF. Also fixes a deadlock in the /release service and bumps effort limits to avoid the underlying overshoot in the first place.

File: pal_pro_gripper_description/robots/pal_pro_gripper.urdf.xacro (robot description, xacro)
@@ -11,4 +11,6 @@
     <xacro:arg name="mj_control" default="false" />
     <xacro:arg name="world_name" default="floor" />
+    <!-- false, true -->
+    <xacro:arg name="calibration_tool" default="False"/>
     <!-- PROPERTIES -->
     <xacro:property name="tool_changer" value="$(arg tool_changer)" />

File: pal_pro_gripper_description/urdf/gripper.ros2_control.xacro (robot description, xacro)
@@ -15,8 +15,24 @@
   <xacro:macro name="ros2_control_pal_pro_gripper" params="name reduction sim_type:=no-simulation">
     <xacro:macro name="ros2_control_pal_pro_gripper_mimic_joint" params="mimic_joint_name actuated_joint_name multiplier sim_type:=no-simulation">
-      <joint name="${mimic_joint_name}">
-        <param name="mimic">${actuated_joint_name}</param>
-        <param name="multiplier">${multiplier}</param>
-      </joint>
+      <xacro:if value="${sim_type == 'gazebo'}">
+        <!-- gz_ros2_control's software mimic controller can drive the joint
+        into its own limit and never recover (unfixed DART bug on Harmonic's
+        dartsim version, see
+        https://github.com/ros-controls/gz_ros2_control/issues/165). Make the
+        joint independently actuated in simulation instead of relying on the
+        URDF mimic tag; the caller is responsible for computing and sending
+        this joint's target position alongside the leader's. -->
+        <joint name="${mimic_joint_name}" mimic="false">
+          <command_interface name="position"/>
+          <state_interface name="position"/>
+        </joint>
+      </xacro:if>
+      <xacro:unless value="${sim_type == 'gazebo'}">
+        <joint name="${mimic_joint_name}">
+          <param name="mimic">${actuated_joint_name}</param>
+          <param name="multiplier">${multiplier}</param>
+          <state_interface name="position"/>
+        </joint>
+      </xacro:unless>
     </xacro:macro>
     <joint name="${name}_finger_joint">
@@ -28,11 +44,11 @@
       <state_interface name="effort"/>
     </joint>
-    <xacro:ros2_control_pal_pro_gripper_mimic_joint mimic_joint_name="${name}_outer_finger_right_joint" actuated_joint_name="${name}_finger_joint" multiplier="-8.28"/>
-    <xacro:ros2_control_pal_pro_gripper_mimic_joint mimic_joint_name="${name}_inner_finger_right_joint" actuated_joint_name="${name}_finger_joint" multiplier="-8.28"/>
-    <xacro:ros2_control_pal_pro_gripper_mimic_joint mimic_joint_name="${name}_fingertip_right_joint" actuated_joint_name="${name}_finger_joint" multiplier="8.28"/>
-    <xacro:ros2_control_pal_pro_gripper_mimic_joint mimic_joint_name="${name}_finger_right_joint" actuated_joint_name="${name}_finger_joint" multiplier="0.22"/>
-    <xacro:ros2_control_pal_pro_gripper_mimic_joint mimic_joint_name="${name}_outer_finger_left_joint" actuated_joint_name="${name}_finger_joint" multiplier="-8.28"/>
-    <xacro:ros2_control_pal_pro_gripper_mimic_joint mimic_joint_name="${name}_inner_finger_left_joint" actuated_joint_name="${name}_finger_joint" multiplier="-8.28"/>
-    <xacro:ros2_control_pal_pro_gripper_mimic_joint mimic_joint_name="${name}_fingertip_left_joint" actuated_joint_name="${name}_finger_joint" multiplier="8.28"/>
+    <xacro:ros2_control_pal_pro_gripper_mimic_joint mimic_joint_name="${name}_outer_finger_right_joint" actuated_joint_name="${name}_finger_joint" multiplier="-8.28" sim_type="${sim_type}"/>
+    <xacro:ros2_control_pal_pro_gripper_mimic_joint mimic_joint_name="${name}_inner_finger_right_joint" actuated_joint_name="${name}_finger_joint" multiplier="-8.28" sim_type="${sim_type}"/>
+    <xacro:ros2_control_pal_pro_gripper_mimic_joint mimic_joint_name="${name}_fingertip_right_joint" actuated_joint_name="${name}_finger_joint" multiplier="8.28" sim_type="${sim_type}"/>
+    <xacro:ros2_control_pal_pro_gripper_mimic_joint mimic_joint_name="${name}_finger_right_joint" actuated_joint_name="${name}_finger_joint" multiplier="0.22" sim_type="${sim_type}"/>
+    <xacro:ros2_control_pal_pro_gripper_mimic_joint mimic_joint_name="${name}_outer_finger_left_joint" actuated_joint_name="${name}_finger_joint" multiplier="-8.28" sim_type="${sim_type}"/>
+    <xacro:ros2_control_pal_pro_gripper_mimic_joint mimic_joint_name="${name}_inner_finger_left_joint" actuated_joint_name="${name}_finger_joint" multiplier="-8.28" sim_type="${sim_type}"/>
+    <xacro:ros2_control_pal_pro_gripper_mimic_joint mimic_joint_name="${name}_fingertip_left_joint" actuated_joint_name="${name}_finger_joint" multiplier="8.28" sim_type="${sim_type}"/>
     <!-- Transmission only set to left finger joint, other joints are passive and mimic this
     joint-->

File: pal_pro_gripper_description/urdf/gripper.urdf.xacro (robot description, xacro)
@@ -13,5 +13,5 @@
       <child link="${name}_screw_${side}_link"/>
       <axis xyz="0 1 0"/>
-      <limit lower="0.0" upper="0.07938" velocity="2" effort="0.1"/>
+      <limit lower="0.0" upper="0.07938" velocity="2" effort="5.0"/>
       <xacro:if value="${side == 'left'}">
         <dynamics damping="0.03"/>
@@ -69,5 +69,5 @@
       <child link="${name}_inner_finger_${side}_link"/>
       <axis xyz="0 0 1"/>
-      <limit lower="${-42.840* deg_to_rad}" upper="${8.001 * deg_to_rad}" velocity="2" effort="0.1"/>
+      <limit lower="${-42.840* deg_to_rad}" upper="${8.001 * deg_to_rad}" velocity="2" effort="5.0"/>
       <mimic joint="${name}_finger_joint" multiplier="-8.28" offset="0.0"/>
     </joint>
@@ -96,5 +96,5 @@
       <child link="${name}_outer_finger_${side}_link"/>
       <axis xyz="0 0 1"/>
-      <limit lower="${-42.840 * deg_to_rad}" upper="${8.001 * deg_to_rad}" velocity="2" effort="0.1"/>
+      <limit lower="${-42.840 * deg_to_rad}" upper="${8.001 * deg_to_rad}" velocity="2" effort="5.0"/>
       <mimic joint="${name}_finger_joint" multiplier="-8.28" offset="0.0"/>
     </joint>
@@ -123,5 +123,5 @@
       <child link="${name}_fingertip_${side}_link"/>
       <axis xyz="0 0 1"/>
-      <limit lower="${-8.001 * deg_to_rad}" upper="${42.840 * deg_to_rad}" velocity="2" effort="0.1"/>
+      <limit lower="${-8.001 * deg_to_rad}" upper="${42.840 * deg_to_rad}" velocity="2" effort="5.0"/>
       <mimic joint="${name}_finger_joint" multiplier="8.28" offset="0.0"/>
     </joint>
