Commit message: Update gazebo launch file and urdf to start simulation

File: pal_pro_gripper_description/gazebo/gazebo.urdf.xacro (robot description, xacro)
@@ -8,35 +8,8 @@
 -->
 <robot name="pal_pro_gripper" xmlns:xacro="http://ros.org/wiki/xacro">
-  <xacro:macro name="mimic_joint_plugin_gazebo" params="name parent_joint mimic_joint has_pid:=false multiplier:=1.0 offset:=0 sensitiveness:=0.0 max_effort:=0.1 robot_namespace:=''">
     <gazebo>
-      <plugin name="${name}_mimic_joint_plugin" filename="libroboticsgroup_upatras_gazebo_mimic_joint_plugin.so">
-        <joint>${parent_joint}</joint>
-        <mimicJoint>${mimic_joint}</mimicJoint>
-        <xacro:if value="${has_pid}">                     <!-- if set to true, PID parameters from "/gazebo_ros_control/pid_gains/${mimic_joint}" are loaded -->
-          <hasPID />
-        </xacro:if>
-        <multiplier>${multiplier}</multiplier>
-        <offset>${offset}</offset>
-        <sensitiveness>${sensitiveness}</sensitiveness>   <!-- if absolute difference between setpoint and process value is below this threshold, do nothing; 0.0 = disable [rad] -->
-        <maxEffort>${max_effort}</maxEffort>              <!-- only taken into account if has_pid:=true [Nm] -->
-        <xacro:unless value="${robot_namespace == ''}">
-          <robotNamespace>${robot_namespace}</robotNamespace>
-        </xacro:unless>
-      </plugin>
+        <plugin name="gazebo_ros_control" filename="libgazebo_ros_control.so">
+            <robotNamespace></robotNamespace>
+        </plugin>
     </gazebo>
-  </xacro:macro>
-  <xacro:macro name="gazebo_gripper_grasp" params="name palm_link finger_link_left finger_link_right ">
-    <gazebo>
-      <gripper name="${name}">
-        <grasp_check>
-          <attach_steps>3</attach_steps>
-          <detach_steps>1</detach_steps>    <!-- should not change otherwise the object will be attached to the gripper too much time -->
-          <min_contact_count>3</min_contact_count>
-        </grasp_check>
-        <gripper_link>${finger_link_left}</gripper_link>
-        <gripper_link>${finger_link_right}</gripper_link>
-        <palm_link>${palm_link}</palm_link>
-      </gripper>
-    </gazebo>
-  </xacro:macro>
 </robot>

File: pal_pro_gripper_description/robots/pal_pro_gripper.urdf.xacro (robot description, xacro)
@@ -4,5 +4,7 @@
     <xacro:property name="name" value="gripper"/>
     <!-- Materials for visualization -->
-    <xacro:include filename="$(find tiago_description)/urdf/materials.urdf.xacro" />
+    <xacro:include filename="$(find pal_pro_gripper_description)/urdf/materials.urdf.xacro" />
+    <!-- Load gazebo plugins -->
+    <xacro:include filename="$(find pal_pro_gripper_description)/gazebo/gazebo.urdf.xacro" />
     <link name="world"/>
     <joint name="world_fixed" type="fixed">

File: pal_pro_gripper_description/urdf/pro_gripper.urdf.xacro (robot description, xacro)
@@ -6,5 +6,5 @@
   <xacro:include filename="$(find pal_pro_gripper_description)/urdf/pro_gripper.transmission.xacro" />
   <!-- Gazebo simulation plugins -->
-  <xacro:include filename="$(find pal_pro_gripper_description)/gazebo/gazebo.urdf.xacro" />
+  <xacro:include filename="$(find pal_pro_gripper_description)/urdf/pro_gripper.gazebo.xacro" />
   <!-- <xacro:include filename="$(find pal_pro_gripper_description)/urdf/grasping_frames.xacro" /> -->
   <xacro:macro name="pro_finger" params="name side reflect">

Commit message: working version of the pal_pro_gripper

File: pal_pro_gripper_description/gazebo/gazebo.urdf.xacro (robot description, xacro)
@@ -18,3 +18,21 @@
         </plugin>
     </gazebo>
+    <xacro:macro name="mimic_joint_plugin_gazebo" params="name parent_joint mimic_joint has_pid:=false multiplier:=1.0 offset:=0 sensitiveness:=0.0 max_effort:=0.1 robot_namespace:=''">
+    <gazebo>
+      <plugin name="${name}_mimic_joint_plugin" filename="libroboticsgroup_upatras_gazebo_mimic_joint_plugin.so">
+        <joint>${parent_joint}</joint>
+        <mimicJoint>${mimic_joint}</mimicJoint>
+        <xacro:if value="${has_pid}">                     <!-- if set to true, PID parameters from "/gazebo_ros_control/pid_gains/${mimic_joint}" are loaded -->
+          <hasPID />
+        </xacro:if>
+        <multiplier>${multiplier}</multiplier>
+        <offset>${offset}</offset>
+        <sensitiveness>${sensitiveness}</sensitiveness>   <!-- if absolute difference between setpoint and process value is below this threshold, do nothing; 0.0 = disable [rad] -->
+        <maxEffort>${max_effort}</maxEffort>              <!-- only taken into account if has_pid:=true [Nm] -->
+        <xacro:unless value="${robot_namespace == ''}">
+          <robotNamespace>${robot_namespace}</robotNamespace>
+        </xacro:unless>
+      </plugin>
+    </gazebo>
+  </xacro:macro>
 </robot>

File: pal_pro_gripper_description/robots/pal_pro_gripper.urdf.xacro (robot description, xacro)
@@ -5,7 +5,11 @@
     <xacro:include filename="$(find pal_urdf_utils)/urdf/materials.urdf.xacro" />
     <xacro:include filename="$(find pal_pro_gripper_description)/urdf/pro_gripper.urdf.xacro" />
-    <xacro:property name="name" value="gripper"/>
     <!-- Load gazebo plugins -->
     <xacro:include filename="$(find pal_pro_gripper_description)/gazebo/gazebo.urdf.xacro" />
+    <xacro:property name="name" value="gripper"/>
+    <xacro:arg name="use_sim" default="false"/>
+    <!-- ros2_control -->
+    <xacro:include filename="$(find pal_pro_gripper_description)/ros2_control/ros2_control.urdf.xacro" />
+    <xacro:pal_pro_gripper_ros2_control use_sim="$(arg use_sim)" />
     <link name="world"/>
     <joint name="world_fixed" type="fixed">

File: pal_pro_gripper_description/urdf/pal_pro_gripper.ros2_control.xacro (robot description, xacro)
@@ -15,4 +15,14 @@
   <xacro:macro name="ros2_control_pal_pro_gripper" params="name reduction" >
     <joint name="${name}_joint">
+      <command_interface name="position"/>
+      <state_interface name="position">
+        <param name="initial_value">0.15</param>
+      </state_interface>
+      <state_interface name="velocity"/>
+      <state_interface name="effort"/>
+    </joint>
+    <joint name="${name}_outer_finger_left_joint">
+      <param name="mimic">${name}_joint</param>
+      <param name="multiplier">1</param>
       <command_interface name="position" />
       <state_interface name="position" />
@@ -20,5 +30,13 @@
       <state_interface name="effort" />
     </joint>
-    <!-- Transmission only set to left outer finger joint, other joints are passive and mimic this
+    <joint name="${name}_outer_finger_right_joint">
+      <param name="mimic">${name}_joint</param>
+      <param name="multiplier">1</param>
+      <command_interface name="position" />
+      <state_interface name="position" />
+      <state_interface name="velocity" />
+      <state_interface name="effort" />
+    </joint>
+    <!-- Transmission only set to left finger joint, other joints are passive and mimic this
     joint-->
     <xacro:include filename="$(find pal_pro_gripper_description)/urdf/pro_gripper.transmission.xacro" />

File: pal_pro_gripper_description/urdf/pro_gripper.urdf.xacro (robot description, xacro)
@@ -3,7 +3,5 @@
   <!--File
   includes-->
-  <!-- Gazebo simulation plugins -->
-  <xacro:include filename="$(find pal_pro_gripper_description)/urdf/pro_gripper.gazebo.xacro" />
-  <!-- <xacro:include filename="$(find pal_pro_gripper_description)/urdf/grasping_frames.xacro" /> -->
+  <!-- TODO: grasping frames -->
   <xacro:macro name="pro_finger" params="name side reflect">
     <link name="${name}_inner_finger_${side}_link">
@@ -40,5 +38,5 @@
     </joint>
     <!-- Mimic finger joint-->
-    <xacro:mimic_joint_plugin_gazebo name="${name}_${side}_mimic_pro_gripper_1"
+     <xacro:mimic_joint_plugin_gazebo name="${name}_${side}_mimic_pro_gripper_1"
       parent_joint="${name}_finger_joint" mimic_joint="${name}_inner_finger_${side}_joint"
       has_pid="false" multiplier="1.0" offset="0" />
@@ -80,7 +78,7 @@
             <dynamics damping="0.03"/>
       </xacro:if>
-      <xacro:unless value="${side == 'left'}">
+      <!-- <xacro:unless value="${side == 'left'}">
             <mimic joint="${name}_finger_joint" multiplier="1" offset="0" />
-      </xacro:unless>
+      </xacro:unless> -->
     </joint>
     <!--  The left outer joint is set as gripper_finger_joint. All other joints are passive and will
@@ -198,5 +196,4 @@
     <xacro:pro_finger name="${name}" side="left" reflect="-1" />
     <xacro:pro_finger name="${name}" side="right" reflect="1" />
-    <xacro:gazebo_gripper_grasp name="${name}_grasp" palm_link="${parent}" finger_link_left="${name}_outer_finger_left_link" finger_link_right="${name}_outer_finger_right_link" />
   </xacro:macro>
 </robot>

Commit message: clean gazebo.urdf.xacro adding gazebo_ros2_control

File: pal_pro_gripper_description/gazebo/gazebo.urdf.xacro (robot description, xacro)
@@ -14,25 +14,7 @@
 <robot name="pal_pro_gripper" xmlns:xacro="http://ros.org/wiki/xacro">
     <gazebo>
-        <plugin name="gazebo_ros2_control" filename="libgazebo_ros2_control.so">
-            <robotNamespace></robotNamespace>
-        </plugin>
-    </gazebo>
-    <xacro:macro name="mimic_joint_plugin_gazebo" params="name parent_joint mimic_joint has_pid:=false multiplier:=1.0 offset:=0 sensitiveness:=0.0 max_effort:=0.1 robot_namespace:=''">
-    <gazebo>
-      <plugin name="${name}_mimic_joint_plugin" filename="libroboticsgroup_upatras_gazebo_mimic_joint_plugin.so">
-        <joint>${parent_joint}</joint>
-        <mimicJoint>${mimic_joint}</mimicJoint>
-        <xacro:if value="${has_pid}">                     <!-- if set to true, PID parameters from "/gazebo_ros_control/pid_gains/${mimic_joint}" are loaded -->
-          <hasPID />
-        </xacro:if>
-        <multiplier>${multiplier}</multiplier>
-        <offset>${offset}</offset>
-        <sensitiveness>${sensitiveness}</sensitiveness>   <!-- if absolute difference between setpoint and process value is below this threshold, do nothing; 0.0 = disable [rad] -->
-        <maxEffort>${max_effort}</maxEffort>              <!-- only taken into account if has_pid:=true [Nm] -->
-        <xacro:unless value="${robot_namespace == ''}">
-          <robotNamespace>${robot_namespace}</robotNamespace>
-        </xacro:unless>
+      <plugin filename="libgazebo_ros2_control.so" name="gazebo_ros2_control">
+        <parameters>$(find pal_pro_gripper_controller_configuration)/config/gazebo_controller_manager_cfg.yaml</parameters>
       </plugin>
     </gazebo>
-  </xacro:macro>
 </robot>

Commit message: update path needed for gz

File: pal_pro_gripper_description/gazebo/gazebo.urdf.xacro (robot description, xacro)
@@ -14,5 +14,5 @@
 <robot name="pal_pro_gripper" xmlns:xacro="http://ros.org/wiki/xacro">
     <gazebo>
-      <plugin filename="libgazebo_ros2_control.so" name="gazebo_ros2_control">
+      <plugin filename="libgz_ros2_control-system.so" name="gz_ros2_control::GazeboSimROS2ControlPlugin">
         <parameters>$(find pal_pro_gripper_controller_configuration)/config/gazebo_controller_manager_cfg.yaml</parameters>
       </plugin>

File: pal_pro_gripper_description/ros2_control/ros2_control.urdf.xacro (robot description, xacro)
@@ -22,5 +22,5 @@
           </xacro:if>
           <xacro:if value="${sim_type == 'gazebo'}">
-            <plugin>gazebo_ros2_control/GazeboSystem</plugin>
+            <plugin>gz_ros2_control/GazeboSimSystem</plugin>
           </xacro:if>
         </xacro:if>

File: pal_pro_gripper_description/urdf/gripper.urdf.xacro (robot description, xacro)
@@ -51,14 +51,14 @@
         <origin xyz="0 0 0" rpy="0 0 0"/>
         <geometry>
-          <mesh filename="package://pal_pro_gripper_description/meshes/inner_finger.stl"/>
-        </geometry>
-        <material name="">
-          <color rgba="0.752941176470588 0.752941176470588 0.752941176470588 1" />
-        </material>
-      </visual>
-      <collision>
-        <origin xyz="0 0 0" rpy="0 0 0"/>
-        <geometry>
-          <mesh filename="package://pal_pro_gripper_description/meshes/inner_finger.stl"/>
+          <mesh filename="file://$(find pal_pro_gripper_description)/meshes/inner_finger.stl"/>
+        </geometry>
+        <material name="">
+          <color rgba="0.752941176470588 0.752941176470588 0.752941176470588 1" />
+        </material>
+      </visual>
+      <collision>
+        <origin xyz="0 0 0" rpy="0 0 0"/>
+        <geometry>
+          <mesh filename="file://$(find pal_pro_gripper_description)/meshes/inner_finger.stl"/>
         </geometry>
       </collision>
@@ -78,14 +78,14 @@
         <origin xyz="0 0 0" rpy="0 0 0"/>
         <geometry>
-          <mesh filename="package://pal_pro_gripper_description/meshes/outer_finger.stl"/>
-        </geometry>
-        <material name="">
-          <color rgba="0.752941176470588 0.752941176470588 0.752941176470588 1" />
-        </material>
-      </visual>
-      <collision>
-        <origin xyz="0 0 0" rpy="0 0 0"/>
-        <geometry>
-          <mesh filename="package://pal_pro_gripper_description/meshes/outer_finger.stl"/>
+          <mesh filename="file://$(find pal_pro_gripper_description)/meshes/outer_finger.stl"/>
+        </geometry>
+        <material name="">
+          <color rgba="0.752941176470588 0.752941176470588 0.752941176470588 1" />
+        </material>
+      </visual>
+      <collision>
+        <origin xyz="0 0 0" rpy="0 0 0"/>
+        <geometry>
+          <mesh filename="file://$(find pal_pro_gripper_description)/meshes/outer_finger.stl"/>
         </geometry>
       </collision>
@@ -105,14 +105,14 @@
         <origin xyz="0 0 0" rpy="0 0 0"/>
         <geometry>
-          <mesh filename="package://pal_pro_gripper_description/meshes/fingertip.stl"/>
-        </geometry>
-        <material name="">
-          <color rgba="0.752941176470588 0.752941176470588 0.752941176470588 1" />
-        </material>
-      </visual>
-      <collision>
-        <origin xyz="0 0 0" rpy="0 0 0"/>
-        <geometry>
-          <mesh filename="package://pal_pro_gripper_description/meshes/fingertip.stl"/>
+          <mesh filename="file://$(find pal_pro_gripper_description)/meshes/fingertip.stl"/>
+        </geometry>
+        <material name="">
+          <color rgba="0.752941176470588 0.752941176470588 0.752941176470588 1" />
+        </material>
+      </visual>
+      <collision>
+        <origin xyz="0 0 0" rpy="0 0 0"/>
+        <geometry>
+          <mesh filename="file://$(find pal_pro_gripper_description)/meshes/fingertip.stl"/>
         </geometry>
       </collision>
@@ -145,5 +145,5 @@
         <origin xyz="0 0 0" rpy="0 0 0" />
         <geometry>
-          <mesh filename="package://pal_pro_gripper_description/meshes/${gripper_base_type}.stl" />
+          <mesh filename="file://$(find pal_pro_gripper_description)/meshes/${gripper_base_type}.stl" />
         </geometry>
         <material name="pal/DarkGrey" />
@@ -152,5 +152,5 @@
         <origin xyz="0 0 0" rpy="0 0 0" />
         <geometry>
-          <mesh filename="package://pal_pro_gripper_description/meshes/${gripper_base_type}.stl" />
+          <mesh filename="file://$(find pal_pro_gripper_description)/meshes/${gripper_base_type}.stl" />
         </geometry>
       </collision>
